File: ESP.kicad_sch (KiCad schematic)
At the start: 13 parts, among them J1 Conn_01x03, SW1 SW_Push, U1 RP2040, U5 W25X40CLSS, U6 DRV8833PW, U7 DRV8833PW, U8 DRV8833PW

Commit message: More progress
Parts:
- removed U6, U7, U8: DRV8833PW, Package_SO:TSSOP-16_4.4x5mm_P0.65mm, symbol Driver_Motor:DRV8833PW
- added J4, J5, J6: Conn_01x12_MountingPin, symbol Connector_Generic_MountingPin:Conn_01x12_MountingPin
- added U6, U7, U8: DRV8835DSSR, DSS0012A, symbol DRV8835:DRV8835DSSR
- added Y1: Resonator, symbol Device:Resonator
Connections:
- net +3.3V: now also J6.1 (Pin_1), J6.11 (Pin_11), J6.3 (Pin_3), J6.5 (Pin_5), J6.7 (Pin_7), J6.9 (Pin_9)
- net Earth: now also J6.10 (Pin_10), J6.12 (Pin_12), J6.2 (Pin_2), J6.4 (Pin_4), J6.6 (Pin_6), J6.8 (Pin_8), U6.13 (GND), U6.6 (GND), U7.13 (GND), U7.6 (GND), U8.13 (GND), U8.6 (GND)
- net Motor_5_A: now reaches U1.11 (GPIO8)
- net Motor_5_A: now also U8.10 (AIN1_APHASE)
- net Motor_5_B: now reaches U1.12 (GPIO9)
- net Motor_5_B: now also U8.9 (AIN2_AENBL)
- net Motor_6_A: now reaches U1.13 (GPIO10)
- net Motor_6_A: now also U1.14 (GPIO11), U8.7 (BIN2_BENBL), U8.8 (BIN1_BPHASE)
- net Motor_1_A: now reaches U1.2 (GPIO0)
- net Motor_1_A: now also U6.10 (AIN1_APHASE)
- net I2C_SCL: now reaches U1.27 (GPIO16)
- net I2C_SDA: now reaches U1.28 (GPIO17)
- net M1_Enc_A: now reaches U1.29 (GPIO18)
- net M1_Enc_A: now also J5.1 (Pin_1)
- net Motor_1_B: now reaches U1.3 (GPIO1)
- net Motor_1_B: now also U6.9 (AIN2_AENBL)
- net M1_Enc_B: now reaches U1.30 (GPIO19)
- net M1_Enc_B: now also J5.2 (Pin_2)
- net M2_Enc_A: now reaches U1.31 (GPIO20)
- net M2_Enc_A: now also J5.3 (Pin_3)
- net M2_Enc_B: now reaches U1.32 (GPIO21)
- net M2_Enc_B: now also J5.4 (Pin_4)
- net M3_Enc_A: now reaches U1.34 (GPIO22)
- net M3_Enc_A: now also J5.5 (Pin_5)
- net M3_Enc_B: now reaches U1.35 (GPIO23)
- net M3_Enc_B: now also J5.6 (Pin_6)
- net M4_Enc_A: now reaches U1.36 (GPIO24)
- net M4_Enc_A: now also J5.7 (Pin_7)
- net M4_Enc_B: now reaches U1.37 (GPIO25)
- net M4_Enc_B: now also J5.8 (Pin_8)
- net M5_Enc_A: now reaches U1.38 (GPIO26_ADC0)
- net M5_Enc_A: now also J5.9 (Pin_9)
- net M5_Enc_B: now reaches U1.39 (GPIO27_ADC1)
- net M5_Enc_B: now also J5.10 (Pin_10)
- net Motor_2_A: now reaches U1.4 (GPIO2)
- net Motor_2_A: now also U6.8 (BIN1_BPHASE)
- net M6_Enc_A: now reaches U1.40 (GPIO28_ADC2)
- net M6_Enc_A: now also J5.11 (Pin_11)
- net M6_Enc_B: now reaches U1.41 (GPIO29_ADC3)
- net M6_Enc_B: now also J5.12 (Pin_12)
- net Motor_2_B: now reaches U1.5 (GPIO3)
- net Motor_2_B: now also U6.7 (BIN2_BENBL)
- net Motor_3_A: now reaches U1.6 (GPIO4)
- net Motor_3_A: now also U7.10 (AIN1_APHASE)
- net Motor_3_B: now reaches U1.7 (GPIO5)
- net Motor_3_B: now also U7.9 (AIN2_AENBL)
- net Motor_4_A: now reaches U1.8 (GPIO6)
- net Motor_4_A: now also U7.8 (BIN1_BPHASE)
- net Motor_4_B: now reaches U1.9 (GPIO7)
- net Motor_4_B: now also U7.7 (BIN2_BENBL)
- new net M1_Out_A: J4.1 (Pin_1), U6.2 (AOUT1)
- new net M1_Out_B: J4.2 (Pin_2), U6.3 (AOUT2)
- new net M2_Out_A: J4.3 (Pin_3), U6.4 (BOUT1)
- new net M2_Out_B: J4.4 (Pin_4), U6.5 (BOUT2)
- new net M3_Out_A: J4.6 (Pin_6), U7.3 (AOUT2)
- new net M3_Out_B: J4.5 (Pin_5), U7.2 (AOUT1)
- new net M4_Out_A: J4.7 (Pin_7), U7.4 (BOUT1)
- new net M4_Out_B: J4.8 (Pin_8), U7.5 (BOUT2)
- new net M5_Out_A: J4.9 (Pin_9), U8.2 (AOUT1)
- new net M5_Out_B: J4.10 (Pin_10), U8.3 (AOUT2)
- new net M6_Out_A: J4.11 (Pin_11), U8.4 (BOUT1)
- new net M6_Out_B: J4.12 (Pin_12), U8.5 (BOUT2)
- new net VCC: U6.12 (VCC), U7.12 (VCC), U8.12 (VCC)
- no-connect marks 0 -> 10
Other:
- note added: "Motor Drivers"
- note added: "Motors Out"
- note added: "SW Debug"
- moved on the sheet: C1, C2, J1, R1, R2, R3, R4, SW1, U1, U5

Commit message: More Progress
Parts:
- removed J4, J5, J6: Conn_01x12_MountingPin, symbol Connector_Generic_MountingPin:Conn_01x12_MountingPin
- removed Y1: Resonator, symbol Device:Resonator
- added C11, C13, C19, C7, C8, C9: 100nF, symbol Device:C_Small
- added C14, C15: 15p, symbol Device:C_Small
- added D4: WS2812B, LED_SMD:LED_WS2812B_PLCC4_5.0x5.0mm_P3.2mm, symbol LED:WS2812B
- added P1, P2, P3, P4, P5, P6: S6B-ZRLFSN, S6B-ZR_JST, symbol JST-ZH:S6B-ZRLFSN
- added R24: 1k, Resistor_SMD:R_0612_1632Metric, symbol Device:R_US
- added SW4: SW_Push, symbol Switch:SW_Push
- added Y1: ABM8G-12.000MHZ-4Y-T3, ABM8G-12.000MHZ-4Y-T3:XTAL_ABM8G-12.000MHZ-4Y-T3, symbol ABMG8_12:ABM8G-12.000MHZ-4Y-T3
- R19: renamed from R3; symbol Device:R -> Device:R_US
- R20: renamed from R4; symbol Device:R -> Device:R_US
- R21: renamed from R2; symbol Device:R -> Device:R_US
- R22: renamed from R1; symbol Device:R -> Device:R_US
- renumbered C1 to C10, C2 to C12, J1 to J4, SW1 to SW2, U5 to U3, U1 to U4, U6 to U5, U7 to U6, U8 to U7
Connections:
- net +3.3V: now also C11.1, C13.1, C19.1, C9.1, P1.2, P2.2, P3.2, P4.2, P5.2, P6.2
- net Earth: now also U4.19 (TESTEN), C14.2, C15.2, D4.3 (VSS), P1.5, P2.5, P3.5, P4.5, P5.5, P6.5, SW4.2, Y1.2 (GND), Y1.4 (GND__1)
- net I2C_SCL: now also U4.18 (GPIO15); no longer U4.27 (GPIO16)
- net I2C_SDA: now also U4.17 (GPIO14); no longer U4.28 (GPIO17)
- net M1_Enc_A: now also P1.3
- net M1_Enc_B: now also P1.4
- net M1_Out_A: now also P1.1
- net M1_Out_B: now also P1.6
- net M2_Enc_A: now also P2.3
- net M2_Enc_B: now also P2.4
- net M2_Out_A: now also P2.1
- net M2_Out_B: now also P2.6
- net M3_Enc_A: now also P3.3
- net M3_Enc_B: now also P3.4
- net M3_Out_A: now also P3.1
- net M3_Out_B: now also P3.6
- net M4_Enc_A: now also P4.3
- net M4_Enc_B: now also P4.4
- net M4_Out_A: now also P4.1
- net M4_Out_B: now also P4.6
- net M5_Enc_A: now also P5.3
- net M5_Enc_B: now also P5.4
- net M5_Out_A: now also P5.1
- net M5_Out_B: now also P5.6
- net M6_Enc_A: now also P6.3
- net M6_Enc_B: now also P6.4
- net M6_Out_A: now also P6.1
- net M6_Out_B: now also P6.6
- net at U4.1 (IOVDD), U4.10 (IOVDD), U4.22 (IOVDD)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: now also C13.2
- net at U4.15 (GPIO12): now also D4.1 (VDD)
- net at U4.16 (GPIO13): now also D4.4 (DIN)
- net XIN: now reaches U4.20 (XIN)
- net XIN: now also C14.1, Y1.1
- net XOUT: now reaches U4.21 (XOUT)
- net XOUT: now also C15.1, Y1.3
- net at U4.23 (DVDD), U4.50 (DVDD): now also C9.2
- net at U4.26 (RUN): now also R24.1
- net at U4.44 (VREG_IN): now also C19.2
- net at U4.48 (USB_VDD): now also C11.2
- new net: R24.2, SW4.1
- new net ESP_PICO_UART_RX: U4.27 (GPIO16)
- new net ESP_PICO_UART_TX: U4.28 (GPIO17)
- no-connect marks 10 -> 5
Other:
- note added: "NeoPixel_Power"
- note added: "Neopixel_Data"
- note added: "Note: No ADC is needed, so the pin is not needed"
- note added: "Reset"
- note added: "Status LED"
- moved on the sheet: U4

Commit message: More progress
Parts:
- removed C7, C8: 100nF, symbol Device:C_Small
- added J4: Conn_01x02, Connector_PinHeader_2.54mm:PinHeader_1x02_P2.54mm_Vertical, symbol Connector_Generic:Conn_01x02
- C10: renamed from C15; footprint (none) -> Capacitor_SMD:C_0402_1005Metric
- C11: renamed from C14; footprint (none) -> Capacitor_SMD:C_0402_1005Metric
- C12: renamed from C10; footprint (none) -> Capacitor_SMD:C_0402_1005Metric
- C13: renamed from C12; footprint (none) -> Capacitor_SMD:C_0402_1005Metric
- C6: renamed from C19; footprint (none) -> Capacitor_SMD:C_0402_1005Metric
- C7: renamed from C11; footprint (none) -> Capacitor_SMD:C_0402_1005Metric
- C8: renamed from C13; footprint (none) -> Capacitor_SMD:C_0402_1005Metric
- C9: footprint (none) -> Capacitor_SMD:C_0402_1005Metric
- P1, P6: value S6B-ZRLFSN -> B6B-ZRLFSN; footprint S6B-ZR_JST -> JST-ZR:CONN_B6B-ZR_JST
- P2: renamed from P4; footprint S6B-ZR_JST -> JST-ZR:CONN_B6B-ZR_JST
- P3: renamed from P2; value S6B-ZRLFSN -> B6B-ZRLFSN; footprint S6B-ZR_JST -> JST-ZR:CONN_B6B-ZR_JST
- P4: renamed from P5; value S6B-ZRLFSN -> B6B-ZRLFSN; footprint S6B-ZR_JST -> JST-ZR:CONN_B6B-ZR_JST
- P5: renamed from P3; value S6B-ZRLFSN -> B6B-ZRLFSN; footprint S6B-ZR_JST -> JST-ZR:CONN_B6B-ZR_JST
- R15: renamed from R19; footprint (none) -> Resistor_SMD:R_0402_1005Metric
- R16: renamed from R20; footprint (none) -> Resistor_SMD:R_0402_1005Metric
- SW2: renamed from SW4; footprint (none) -> Button_Switch_SMD:SW_SPST_PTS645
- SW3: renamed from SW2; footprint (none) -> Button_Switch_SMD:SW_SPST_PTS645
- U3: renamed from U5; footprint DSS0012A -> DRV8835:DSS0012A
- U5: renamed from U6; footprint DSS0012A -> DRV8835:DSS0012A
- U6: renamed from U7; footprint DSS0012A -> DRV8835:DSS0012A
- Y1: footprint ABM8G-12.000MHZ-4Y-T3:XTAL_ABM8G-12.000MHZ-4Y-T3 -> ABM8G:XTAL_ABM8G-12.000MHZ-4Y-T3
- renumbered D4 to D5, J4 to J5, R24 to R14, R21 to R17, R22 to R18, U3 to U7
Connections:
- net +3.3V: now also U3.12 (VCC), U5.12 (VCC)
- net Earth: now also U4.45 (VREG_VOUT)
- net I2C_SCL: now also J4.2 (Pin_2)
- net I2C_SDA: now also J4.1 (Pin_1)
- net VCC: now also U3.1 (VM), U5.1 (VM), U6.1 (VM); no longer U3.12 (VCC), U5.12 (VCC)
- net at U4.15 (GPIO12): no longer D5.1 (VDD)
- net ESP_PICO_UART_RX renamed PICO_UART_TX
- net ESP_PICO_UART_TX renamed PICO_UART_RX
- net USB_DM_1 renamed USB_DP_Pico
- net USB_DP_1 renamed USB_DM_Pico
- new net +5V: D5.1 (VDD)
- no-connect marks 5 -> 6
Other:
- added sheet IMU (ICM_20984.kicad_sch)
- note added: "I2C Access Point"
- note added: "PICO RX"
- note added: "PICO TX"
- note removed: "NeoPixel_Power"
- moved on the sheet: D5

Commit message: Nearly done schematics
Parts:
- removed R14: 1k, Resistor_SMD:R_0612_1632Metric, symbol Device:R_US
- removed SW2: SW_Push, Button_Switch_SMD:SW_SPST_PTS645, symbol Switch:SW_Push
- SW3: footprint Button_Switch_SMD:SW_SPST_PTS645 -> Button_Switch_SMD:SW_SPST_PTS810
- U3, U5, U6: footprint DRV8835:DSS0012A -> Package_SON:WSON-12-1EP_3x2mm_P0.5mm_EP1x2.65_ThermalVias
- renumbered C9 to C10, C10 to C11, C11 to C12, C12 to C13, C13 to C14, C6 to C7, C7 to C8, C8 to C9, P3 to P2, P5 to P3, P2 to P4, P4 to P5
Connections:
- net +3.3V: now also U6.12 (VCC)
- net I2C_SCL: now also U4.28 (GPIO17); no longer U4.18 (GPIO15)
- net I2C_SDA: now also U4.27 (GPIO16); no longer U4.17 (GPIO14)
- net M1_Out_A: now also U3.5 (BOUT2); no longer U3.2 (AOUT1)
- net M1_Out_B: now also U3.4 (BOUT1); no longer U3.3 (AOUT2)
- net M2_Out_A: now also U3.2 (AOUT1); no longer U3.4 (BOUT1)
- net M2_Out_B: now also U3.3 (AOUT2); no longer U3.5 (BOUT2)
- net M3_Out_A: now also U5.5 (BOUT2); no longer U5.3 (AOUT2)
- net M3_Out_B: now also U5.4 (BOUT1); no longer U5.2 (AOUT1)
- net M4_Out_A: now also U5.2 (AOUT1); no longer U5.4 (BOUT1)
- net M4_Out_B: now also U5.3 (AOUT2); no longer U5.5 (BOUT2)
- net M5_Out_A: now also U6.5 (BOUT2); no longer U6.2 (AOUT1)
- net M5_Out_B: now also U6.4 (BOUT1); no longer U6.3 (AOUT2)
- net M6_Out_A: now also U6.2 (AOUT1); no longer U6.4 (BOUT1)
- net M6_Out_B: now also U6.3 (AOUT2); no longer U6.5 (BOUT2)
- net Motor_1_A: now also U3.7 (BIN2_BENBL), U4.14 (GPIO11); no longer U3.10 (AIN1_APHASE), U4.2 (GPIO0)
- net Motor_1_B: now also U3.8 (BIN1_BPHASE), U4.13 (GPIO10); no longer U3.9 (AIN2_AENBL), U4.3 (GPIO1)
- net Motor_2_A: now also U3.10 (AIN1_APHASE), U4.11 (GPIO8); no longer U3.8 (BIN1_BPHASE), U4.4 (GPIO2)
- net Motor_2_B: now also U3.9 (AIN2_AENBL), U4.12 (GPIO9); no longer U3.7 (BIN2_BENBL), U4.5 (GPIO3)
- net Motor_3_A: now also U4.9 (GPIO7), U5.7 (BIN2_BENBL); no longer U4.6 (GPIO4), U5.10 (AIN1_APHASE)
- net Motor_3_B: now also U4.8 (GPIO6), U5.8 (BIN1_BPHASE); no longer U4.7 (GPIO5), U5.9 (AIN2_AENBL)
- net Motor_4_A: now also U4.6 (GPIO4), U5.10 (AIN1_APHASE); no longer U4.8 (GPIO6), U5.8 (BIN1_BPHASE)
- net Motor_4_B: now also U4.7 (GPIO5), U5.9 (AIN2_AENBL); no longer U4.9 (GPIO7), U5.7 (BIN2_BENBL)
- net Motor_5_A: now also U4.5 (GPIO3), U6.7 (BIN2_BENBL); no longer U4.11 (GPIO8), U6.10 (AIN1_APHASE)
- net Motor_5_B: now also U4.4 (GPIO2), U6.8 (BIN1_BPHASE); no longer U4.12 (GPIO9), U6.9 (AIN2_AENBL)
- net Motor_6_A: now also U4.2 (GPIO0), U6.10 (AIN1_APHASE); no longer U4.13 (GPIO10), U4.14 (GPIO11), U6.7 (BIN2_BENBL), U6.8 (BIN1_BPHASE)
- net PICO_UART_RX: now also U4.17 (GPIO14); no longer U4.28 (GPIO17)
- net PICO_UART_TX: now also U4.16 (GPIO13); no longer U4.27 (GPIO16)
- net VCC: no longer U6.12 (VCC)
- net at D5.4 (DIN): now also U4.18 (GPIO15); no longer U4.16 (GPIO13)
- net Pico_PU: now reaches U4.26 (RUN)
- new net Motor_6_B: U4.3 (GPIO1), U6.9 (AIN2_AENBL)
Other:
- note removed: "Reset"
- moved on the sheet: D5, P2, P3, P4, P5

Commit message: Much much more progress
Parts:
- removed J4: Conn_01x02, Connector_PinHeader_2.54mm:PinHeader_1x02_P2.54mm_Vertical, symbol Connector_Generic:Conn_01x02
- added C33: 100nF, Capacitor_SMD:C_0402_1005Metric, symbol Device:C_Small
- added J5: B4B-ZRLFSN, JST-ZR-4Pin:CONN_B4B-ZRLFSN_JST, symbol JST-ZH-4Pin:B4B-ZRLFSN
- R18: footprint Resistor_SMD:R_0612_1632Metric -> Resistor_SMD:R_0402_1005Metric
- renumbered SW3 to Boot1, J5 to SWD1
Connections:
- net +3.3V: now also J5.1
- net +5V: now also C33.2
- net Earth: now also C33.1, J5.4
- net I2C_SCL: now also J5.3
- net I2C_SDA: now also J5.2
- net M1_Enc_A: now also U4.30 (GPIO19); no longer U4.29 (GPIO18)
- net M1_Enc_B: now also U4.29 (GPIO18); no longer U4.30 (GPIO19)
- net ESP_RX: now reaches U4.15 (GPIO12)
- net PICO_UART_RX: no longer names the net of U4.17 (GPIO14)
- net PICO_UART_TX renamed ESP_TX

Commit message: Rev 1
Parts:
- added C35, C41: 1uf, Capacitor_SMD:C_0201_0603Metric, symbol Device:C_Small
- added C36, C37, C38, C39, C40, C42: 100nF, Capacitor_SMD:C_0201_0603Metric, symbol Device:C_Small
- C10, C7, C8, C9: footprint Capacitor_SMD:C_0402_1005Metric -> Capacitor_SMD:C_0201_0603Metric
- R17: footprint Resistor_SMD:R_0612_1632Metric -> Resistor_SMD:R_0603_1608Metric_Pad0.98x0.95mm_HandSolder; now not fitted
Connections:
- net +3.3V: now also C9.2, U4.1 (IOVDD), U4.10 (IOVDD), U4.22 (IOVDD), U4.33 (IOVDD), U4.42 (IOVDD), U4.43 (ADC_AVDD), U4.44 (VREG_IN), U4.48 (USB_VDD), U4.49 (IOVDD), C36.2, C37.2, C38.2, C39.1, C40.2, C41.2; no longer C10.1, C9.1, J5.1
- net +5V: now also J5.1
- net Earth: now also C10.2, C7.2, C8.2, C9.1, C35.2, C36.1, C37.1, C38.1, C39.2, C40.1, C41.1, C42.2; no longer U4.45 (VREG_VOUT)
- net at U4.23 (DVDD), U4.50 (DVDD): now also C10.1, U4.45 (VREG_VOUT), C35.1, C42.1; no longer C10.2
- no-connect marks 6 -> 5
Other:
- moved on the sheet: C10, C7, C8, C9

Commit message: Rev0.1
Parts:
- C8: Name (none) -> C40
Connections:
- net I2C_SCL renamed PICO_SCL
- net I2C_SDA renamed PICO_SDA
Changed lines of the file:
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@@
   (junction (at 266.7 106.68) (diameter 0) (color 0 0 0 0)
   )
-  (junction (at 161.544 26.67) (diameter 0) (color 0 0 0 0)
+  (junction (at 161.544 25.908) (diameter 0) (color 0 0 0 0)
   )
   (junction (at 59.563 29.845) (diameter 0) (color 0 0 0 0)
@@
     (stroke (width 0) (type default))
   )
-  (wire (pts (xy 159.766 28.448) (xy 160.274 28.448))
+  (wire (pts (xy 159.131 28.448) (xy 160.274 28.448))
+    (stroke (width 0) (type default))
+  )
+  (polyline (pts (xy 144.526 58.293) (xy 144.526 58.547))
     (stroke (width 0) (type default))
   )
@@
     (stroke (width 0) (type default))
   )
+  (polyline (pts (xy 150.495 58.547) (xy 144.526 58.547))
+    (stroke (width 0) (type default))
+  )
   (wire (pts (xy 140.335 179.705) (xy 146.685 179.705))
     (stroke (width 0) (type default))
@@
     (stroke (width 0) (type default))
   )
-  (wire (pts (xy 159.766 26.67) (xy 161.544 26.67))
+  (wire (pts (xy 159.131 25.908) (xy 161.544 25.908))
     (stroke (width 0) (type default))
   )
@@
     (stroke (width 0) (type default))
   )
-  (wire (pts (xy 104.14 81.915) (xy 96.52 81.915))
+  (wire (pts (xy 115.316 81.915) (xy 96.52 81.915))
     (stroke (width 0) (type default))
   )
@@
     (stroke (width 0) (type default))
   )
-  (polyline (pts (xy 150.495 12.065) (xy 150.495 58.42))
+  (polyline (pts (xy 144.526 12.192) (xy 144.526 58.547))
     (stroke (width 0) (type default))
   )
-  (wire (pts (xy 161.544 26.67) (xy 161.544 44.196))
+  (wire (pts (xy 161.544 25.908) (xy 161.544 44.196))
     (stroke (width 0) (type default))
   )
@@
     (stroke (width 0) (type default))
   )
-  (wire (pts (xy 161.544 26.67) (xy 177.292 26.67))
+  (wire (pts (xy 161.544 25.908) (xy 177.292 25.908))
     (stroke (width 0) (type default))
   )
@@
     (stroke (width 0) (type default))
   )
-  (wire (pts (xy 104.14 84.455) (xy 96.52 84.455))
+  (wire (pts (xy 115.316 84.455) (xy 96.52 84.455))
     (stroke (width 0) (type default))
   )
@@
     (fill (type none))
   )
-  (rectangle (start 150.495 58.42) (end 206.375 93.98)
+  (rectangle (start 150.495 58.547) (end 206.375 94.107)
     (stroke (width 0) (type default))
     (fill (type none))
@@
     (effects (font (size 1.27 1.27)) (justify left bottom))
   )
-  (label "I2C_SCL" (at 104.14 84.455 0) (fields_autoplaced)
-    (effects (font (size 1.27 1.27)) (justify left bottom))
-  )
   (label "M6_Out_A" (at 271.78 125.73 0) (fields_autoplaced)
     (effects (font (size 1.27 1.27)) (justify left bottom))
@@
     (effects (font (size 1.27 1.27)) (justify left bottom))
   )
-  (label "I2C_SDA" (at 104.14 81.915 0) (fields_autoplaced)
-    (effects (font (size 1.27 1.27)) (justify left bottom))
-  )
   (label "M4_Out_A" (at 270.51 81.28 0) (fields_autoplaced)
     (effects (font (size 1.27 1.27)) (justify left bottom))
@@
     (effects (font (size 1.27 1.27)) (justify right bottom))
   )
-  (label "I2C_SDA" (at 159.766 26.67 180) (fields_autoplaced)
-    (effects (font (size 1.27 1.27)) (justify right bottom))
-  )
   (label "M2_Out_A" (at 182.245 102.87 180) (fields_autoplaced)
     (effects (font (size 1.27 1.27)) (justify right bottom))
@@
     (effects (font (size 1.27 1.27)) (justify right bottom))
   )
-  (label "I2C_SCL" (at 159.766 28.448 180) (fields_autoplaced)
-    (effects (font (size 1.27 1.27)) (justify right bottom))
-  )
   (label "XIN" (at 33.655 94.615 180) (fields_autoplaced)
     (effects (font (size 1.27 1.27)) (justify right bottom))
@@
     )
   )
+  (global_label "PICO_SDA" (shape input) (at 159.131 25.908 180) (fields_autoplaced)
+    (effects (font (size 1.27 1.27)) (justify right))
+    (property "Intersheetrefs" "${INTERSHEET_REFS}" (at 147.1348 25.908 0)
+      (effects (font (size 1.27 1.27)) (justify right) hide)
+    )
+  )
+  (global_label "PICO_SDA" (shape input) (at 115.316 81.915 0) (fields_autoplaced)
+    (effects (font (size 1.27 1.27)) (justify left))
+    (property "Intersheetrefs" "${INTERSHEET_REFS}" (at 127.3122 81.915 0)
+      (effects (font (size 1.27 1.27)) (justify left) hide)
+    )
+  )
   (global_label "ESP_TX" (shape input) (at 106.045 74.295 0) (fields_autoplaced)
     (effects (font (size 1.27 1.27)) (justify left))
@@
     )
   )
+  (global_label "PICO_SCL" (shape input) (at 159.131 28.448 180) (fields_autoplaced)
+    (effects (font (size 1.27 1.27)) (justify right))
+    (property "Intersheetrefs" "${INTERSHEET_REFS}" (at 147.1953 28.448 0)
+      (effects (font (size 1.27 1.27)) (justify right) hide)
+    )
+  )
+  (global_label "PICO_SCL" (shape input) (at 115.316 84.455 0) (fields_autoplaced)
+    (effects (font (size 1.27 1.27)) (justify left))
+    (property "Intersheetrefs" "${INTERSHEET_REFS}" (at 127.2517 84.455 0)
+      (effects (font (size 1.27 1.27)) (justify left) hide)
+    )
+  )
   (hierarchical_label "Pico_PU" (shape input) (at 30.48 41.275 180) (fields_autoplaced)
     (effects (font (size 1.27 1.27)) (justify right))
@@
   )
   (symbol (lib_id "Device:C_Small") (at 85.09 24.638 0) (unit 1)
-    (in_bom yes) (on_board yes) (dnp no) (fields_autoplaced)
+    (in_bom yes) (on_board no) (dnp no)
     (property "Reference" "C8" (at 87.63 23.3743 0)
-      (effects (font (size 1.27 1.27)) (justify left))
+      (effects (font (size 1.27 1.27)) (justify left) hide)
     )
     (property "Value" "100nF" (at 87.63 25.9143 0)
@@
       (effects (font (size 1.27 1.27)) hide)
     )
+    (property "Sim.Enable" "0" (at 85.09 24.638 0)
+      (effects (font (size 1.27 1.27)) hide)
+    )
+    (property "Name" "C40" (at 90.424 24.003 0)
+      (effects (font (size 1.27 1.27)))
+    )
     (pin "1")
     (pin "2")
@@
       (effects (font (size 1.27 1.27)) (justify left top))
     )
-    (pin "Pico_SDA" bidirectional (at 177.292 26.67 180)
+    (pin "Pico_SDA" bidirectional (at 177.292 25.908 180)
       (effects (font (size 1.27 1.27)) (justify left))
     )
