File: DeltaRhoRobot.kicad_pcb (KiCad board)
At the start: 4 copper layers, 76.2 x 76.2 mm, 107 parts, among them J1 Conn_01x02_Socket, J10 Conn_01x02, J11 Conn_01x07, J12 USB_C_Receptacle_USB2.0, J2 USB_C_Receptacle_USB2.0, J3 USB_C_Receptacle_USB2.0, J4 Conn_01x02, J5 Conn_01x03, J6 Conn_02x20_Counter_Clockwise, J7 Conn_01x08, J8 Conn_01x08, J9 Conn_01x04, P1 B6B-ZRLFSN, P2 S6B-ZRLFSN, P3 B6B-ZRLFSN, P4 B6B-ZRLFSN, P5 B6B-ZRLFSN, P6 B6B-ZRLFSN, Q1 MBT3904DW1, Q2 DMN65D8L, Q4 DMN65D8L, SW1 CAS-120A1, SW2 SW_Push, SW3 SW_Push, SW4 SW_Push, SW5 SW_Push, SW6 SW_Push, U1 AP63205WU-7, U10 ICM-20948, U11 FT231XS, U12 ESP32-CAM, U2 AMS1117-3.3, U3 DRV8835DSSR, U4 RP2040, U5 DRV8835DSSR, U6 DRV8835DSSR, U7 W25X40CLSS, U8 ESP32-S3-WROOM-1-N8R2, U9 AMS1117-1.8, Y1 ABM8G-12.000MHZ-4Y-T3

Commit message: Nearly done schematics
Parts:
- added C29: 0.1uF, Capacitor_SMD:C_0402_1005Metric, F.Cu at (145.1, 39.2)
- added J13: Conn_02x09_Top_Bottom, Connector_PinSocket_2.54mm:PinSocket_2x09_P2.54mm_Vertical, F.Cu at (165.5, 52.9)
- added Q3: STB55NF06T4, Package_TO_SOT_SMD:TO-263-2, F.Cu at (168.6, 109.7)
- added R32: 68k, Resistor_SMD:R_0402_1005Metric, F.Cu at (167.5, 118.3)
- added REF**: MountingHole_3.2mm_M3_ISO14580_Pad_TopOnly, MountingHole:MountingHole_3.2mm_M3_ISO14580_Pad_TopOnly, F.Cu at (155.0, 55.0)
- added REF**: MountingHole_3.2mm_M3_ISO14580_Pad_TopOnly, MountingHole:MountingHole_3.2mm_M3_ISO14580_Pad_TopOnly, F.Cu at (220.0, 120.0)
- added REF**: MountingHole_3.2mm_M3_ISO14580_Pad_TopOnly, MountingHole:MountingHole_3.2mm_M3_ISO14580_Pad_TopOnly, F.Cu at (220.0, 55.0)
- added REF**: MountingHole_3.2mm_M3_ISO14580_Pad_TopOnly, MountingHole:MountingHole_3.2mm_M3_ISO14580_Pad_TopOnly, F.Cu at (155.0, 120.0)
- C10: value 15p -> 100nF
- C12: value 2.2u -> 15p
- C13: value 100n -> 2.2u
- C14: value 22uf -> 100n
- C17: value 0.1uF -> 22uf
- C22: value 0.1uf -> 0.1uF
- C24: value 10uF -> 0.1uf
- C25: value 47pF -> 10uF
- C27: value 0.1uF -> 47pF
- C4: value C_Small -> 10uF
- C6: value 100nF -> 10uF
- D1: value 1N5820 -> SS34; footprint Diode_THT:D_DO-201AD_P15.24mm_Horizontal -> Diode_SMD:D_SOD-123
- J6: value Conn_02x20_Counter_Clockwise -> Conn_01x09; footprint Connector_PinSocket_2.54mm:PinSocket_2x20_P2.54mm_Vertical -> Connector_PinSocket_2.54mm:PinSocket_1x09_P2.54mm_Vertical
- J7: value Conn_01x08 -> Conn_02x20_Counter_Clockwise; footprint Connector_PinSocket_2.54mm:PinSocket_1x08_P2.54mm_Vertical -> Connector_PinSocket_2.54mm:PinSocket_2x20_P2.54mm_Vertical
- J9: value Conn_01x04 -> Conn_01x08; footprint Connector_PinSocket_2.54mm:PinSocket_1x04_P2.54mm_Vertical -> Connector_PinSocket_2.54mm:PinSocket_1x08_P2.54mm_Vertical
- SW1: footprint Button_Switch_SMD:Nidec_Copal_CAS-120A -> switch185:1825232-1_TEC
- SW3, SW4: footprint Button_Switch_SMD:SW_SPST_PTS645 -> Button_Switch_SMD:SW_SPST_PTS810
- U2: footprint Package_SO:SOIC-8_3.9x4.9mm_P1.27mm -> Package_TO_SOT_SMD:SOT-223-3_TabPin2
- U3, U5, U6: footprint DRV8835:DSS0012A -> Package_SON:WSON-12-1EP_3x2mm_P0.5mm_EP1x2.65_ThermalVias
- moved SW5 286.5 mm to (332.5, 63.0)
- moved J8 283.5 mm to (312.2, 94.9)
- moved R29 282.0 mm to (330.6, 103.1), turned to 90 degrees
- moved R30 279.5 mm to (328.4, 103.1)
- moved R25 279.3 mm to (330.2, 94.6), turned to 180 degrees
- moved C27 278.0 mm to (330.6, 105.0), turned to -90 degrees
- moved C26 276.0 mm to (328.2, 104.5), turned to 180 degrees
- moved C28 272.3 mm to (327.7, 84.1)
- moved R31 270.9 mm to (315.9, 109.9), turned to 180 degrees
- moved R28 267.1 mm to (317.1, 100.2), turned to 180 degrees
- moved C10 205.8 mm to (241.1, 103.1), turned to 90 degrees
- moved D1 186.6 mm to (239.6, 94.9), turned to 90 degrees
- moved SW4 173.1 mm to (218.1, 42.7), turned to 90 degrees
- moved C24 169.9 mm to (183.0, 167.2)
- moved C25 169.9 mm to (183.0, 159.3)
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- renumbered P3 to P2, P5 to P3, P2 to P4, P4 to P5
Connections:
- C10 pad 1: /Pico/XOUT -> +3.3V
- C10 pad 2: Earth -> Net-(C10-Pad2)
- C11 pad 1: /Pico/XIN -> /Pico/XOUT
- C12 pad 1: +3.3V -> /Pico/XIN
- C14 pad 1: Net-(U8-3V3) -> +3.3V
- C15 pad 2: Net-(U8-3V3) -> +3.3V
- C16 pad 2: Net-(U8-3V3) -> +3.3V
- C17 pad 2: Net-(U8-GPIO0/BOOT) -> +3.3V
- C18 pad 2: /ESP32-S3-WROOM-1/ADC3 -> Net-(U8-GPIO0/BOOT)
- C19 pad 2: /ESP32-S3-WROOM-1/ADC2 -> /ESP32-S3-WROOM-1/ADC0
- C21 pad 2: /ESP32-S3-WROOM-1/ADC0 -> /ESP32-S3-WROOM-1/ADC2
- C22 pad 1: +3.3V -> Earth
- C22 pad 2: Earth -> /ESP32-S3-WROOM-1/ADC3
- C23 pad 1: Net-(U10-REGOUT) -> +3.3V
- C24 pad 1: /ESP32-S3-WROOM-1/ESP32CAM/V_USB -> Net-(U10-REGOUT)
- C25 pad 1: /ESP32-S3-WROOM-1/ESP32CAM/ESPCAM_USB_D+ -> /ESP32-S3-WROOM-1/ESP32CAM/V_USB
- C26 pad 1: /ESP32-S3-WROOM-1/ESP32CAM/ESPCAM_USB_D- -> /ESP32-S3-WROOM-1/ESP32CAM/ESPCAM_USB_D+
- C27 pad 1: /ESP32-S3-WROOM-1/ESP32CAM/3.3V_Out -> /ESP32-S3-WROOM-1/ESP32CAM/ESPCAM_USB_D-
- C28 pad 1: Earth -> /ESP32-S3-WROOM-1/ESP32CAM/3.3V_Out
- C28 pad 2: Net-(U12-GPIO0) -> Earth
- C3 pad 1: Net-(SW1-A) -> Net-(Q3-S)
- C6 pad 1: +3.3V -> Net-(C6-Pad1)
- C6 pad 2: Net-(U4-VREG_IN) -> Earth
- C7 pad 2: Net-(U4-USB_VDD) -> Net-(U4-VREG_IN)
- C8 pad 2: Net-(C8-Pad2) -> Net-(U4-USB_VDD)
- D2 pad 3: Net-(D1-K) -> Net-(Q3-S)
- J6 pad 1: unconnected-(J6-Pin_1-Pad1) -> /ESP32-S3-WROOM-1/ADC0
- J6 pad 2: unconnected-(J6-Pin_2-Pad2) -> /ESP32-S3-WROOM-1/ADC1
- J6 pad 3: unconnected-(J6-Pin_3-Pad3) -> /ESP32-S3-WROOM-1/ADC2
- J6 pad 4: unconnected-(J6-Pin_4-Pad4) -> /ESP32-S3-WROOM-1/ADC3
- J6 pad 5: unconnected-(J6-Pin_5-Pad5) -> /ESP32-S3-WROOM-1/GPIO_15
- J6 pad 6: unconnected-(J6-Pin_6-Pad6) -> /ESP32-S3-WROOM-1/GPIO_16
- J6 pad 7: unconnected-(J6-Pin_7-Pad7) -> /ESP32-S3-WROOM-1/GPIO_17
- J6 pad 8: unconnected-(J6-Pin_8-Pad8) -> /ESP32-S3-WROOM-1/GPIO_18
- J6 pad 9: unconnected-(J6-Pin_9-Pad9) -> /ESP32-S3-WROOM-1/GPIO_8
- J7 pad 1: Earth -> unconnected-(J7-Pin_1-Pad1)
- J7 pad 5: Earth -> unconnected-(J7-Pin_5-Pad5)
- J7 pad 8: +3.3V -> unconnected-(J7-Pin_8-Pad8)
- J8 pad 1: unconnected-(J8-Pin_1-Pad1) -> Earth
- J8 pad 2: /ESP32-S3-WROOM-1/Handshake -> unconnected-(J8-Pin_2-Pad2)
- J8 pad 3: /ESP32-S3-WROOM-1/ESP_SCLK -> unconnected-(J8-Pin_3-Pad3)
- J8 pad 4: /ESP32-S3-WROOM-1/ESP_CS0 -> unconnected-(J8-Pin_4-Pad4)
- J8 pad 5: /ESP32-S3-WROOM-1/ESP_MOSI -> Earth
- J8 pad 6: /ESP32-S3-WROOM-1/ESP_MISO -> unconnected-(J8-Pin_6-Pad6)
- J8 pad 7: Earth -> unconnected-(J8-Pin_7-Pad7)
- J8 pad 8: unconnected-(J8-Pin_8-Pad8) -> +3.3V
- J9 pad 1: /ESP32-S3-WROOM-1/ADC3 -> unconnected-(J9-Pin_1-Pad1)
- J9 pad 2: /ESP32-S3-WROOM-1/ADC2 -> /ESP32-S3-WROOM-1/Handshake
- J9 pad 3: /ESP32-S3-WROOM-1/ADC1 -> /ESP32-S3-WROOM-1/ESP_SCLK
- J9 pad 4: /ESP32-S3-WROOM-1/ADC0 -> /ESP32-S3-WROOM-1/ESP_CS0
- R14 pad 2: Net-(R14-Pad2) -> +3.3V
- R19 pad 1: Net-(U8-3V3) -> Net-(U8-EN)
- R29 pad 2: /ESP32-S3-WROOM-1/ESP32CAM/3.3V_Out -> Net-(U11-USBDM)
- R30 pad 1: /ESP32-S3-WROOM-1/ESP32CAM/3.3V_Out -> Net-(U11-USBDP)
- R4 pad 2: Net-(C5-Pad1) -> Net-(C6-Pad1)
- R7 pad 1: Net-(C5-Pad1) -> Net-(C6-Pad1)
- R8 pad 1: Net-(C5-Pad1) -> Net-(C6-Pad1)
- SW1 pad 1: unconnected-(SW1-C-Pad1) -> Net-(SW1-A)
- SW1 pad 2: Net-(D1-K) -> Net-(Q3-G)
- SW1 pad 3: Net-(SW1-A) -> Earth
- SW2 pad 1: Net-(R14-Pad2) -> +3.3V
- SW4 pad 1: Earth -> Net-(U8-GPIO0/BOOT)
- SW4 pad 2: Net-(U8-3V3) -> Earth
- SW5 pad 1: Net-(U8-GPIO0/BOOT) -> Net-(U12-GPIO0)
- U1 pad 2: Net-(SW1-A) -> Net-(Q3-S)
- U1 pad 3: Net-(SW1-A) -> Net-(Q3-S)
- U11 pad 11: /ESP32-S3-WROOM-1/ESP32CAM/3.3V_Out -> Net-(U11-USBDP)
- U11 pad 12: /ESP32-S3-WROOM-1/ESP32CAM/3.3V_Out -> Net-(U11-USBDM)
- U2 pad 3: Net-(SW1-A) -> Net-(Q3-S)
- U3 pad 10: /Pico/Motor_1_A -> /Pico/Motor_2_A
- U3 pad 2: /Pico/M1_Out_A -> /Pico/M2_Out_A
- U3 pad 3: /Pico/M1_Out_B -> /Pico/M2_Out_B
- U3 pad 4: /Pico/M2_Out_A -> /Pico/M1_Out_B
- U3 pad 5: /Pico/M2_Out_B -> /Pico/M1_Out_A
- U3 pad 7: /Pico/Motor_2_B -> /Pico/Motor_1_A
- U3 pad 8: /Pico/Motor_2_A -> /Pico/Motor_1_B
- U3 pad 9: /Pico/Motor_1_B -> /Pico/Motor_2_B
- U4 pad 1: Net-(C8-Pad2) -> Net-(C9-Pad2)
- U4 pad 10: Net-(C8-Pad2) -> Net-(C9-Pad2)
- U4 pad 11: /Pico/Motor_5_A -> /Pico/Motor_2_A
- U4 pad 12: /Pico/Motor_5_B -> /Pico/Motor_2_B
- U4 pad 13: /Pico/Motor_6_A -> /Pico/Motor_1_B
- U4 pad 14: /Pico/Motor_6_A -> /Pico/Motor_1_A
- U4 pad 16: Net-(D5-DIN) -> /ESP_PICO_UART_RX
- U4 pad 17: /Pico/I2C_SDA -> /ESP_PICO_UART_TX
- U4 pad 18: /Pico/I2C_SCL -> Net-(D5-DIN)
- U4 pad 2: /Pico/Motor_1_A -> /Pico/Motor_6_A
- U4 pad 22: Net-(C8-Pad2) -> Net-(C9-Pad2)
- U4 pad 23: Net-(C9-Pad2) -> Net-(C10-Pad2)
- U4 pad 27: /ESP_PICO_UART_RX -> /Pico/I2C_SDA
- U4 pad 28: /ESP_PICO_UART_TX -> /Pico/I2C_SCL
- U4 pad 3: /Pico/Motor_1_B -> /Pico/Motor_6_B
- U4 pad 33: Net-(C8-Pad2) -> Net-(C9-Pad2)
- U4 pad 4: /Pico/Motor_2_A -> /Pico/Motor_5_B
- U4 pad 42: Net-(C8-Pad2) -> Net-(C9-Pad2)
- U4 pad 49: Net-(C8-Pad2) -> Net-(C9-Pad2)
- U4 pad 5: /Pico/Motor_2_B -> /Pico/Motor_5_A
- U4 pad 50: Net-(C9-Pad2) -> Net-(C10-Pad2)
- U4 pad 6: /Pico/Motor_3_A -> /Pico/Motor_4_A
- U4 pad 7: /Pico/Motor_3_B -> /Pico/Motor_4_B
- U4 pad 8: /Pico/Motor_4_A -> /Pico/Motor_3_B
- U4 pad 9: /Pico/Motor_4_B -> /Pico/Motor_3_A
- U5 pad 10: /Pico/Motor_3_A -> /Pico/Motor_4_A
- U5 pad 2: /Pico/M3_Out_B -> /Pico/M4_Out_A
- U5 pad 3: /Pico/M3_Out_A -> /Pico/M4_Out_B
- U5 pad 4: /Pico/M4_Out_A -> /Pico/M3_Out_B
- U5 pad 5: /Pico/M4_Out_B -> /Pico/M3_Out_A
- U5 pad 7: /Pico/Motor_4_B -> /Pico/Motor_3_A
- U5 pad 8: /Pico/Motor_4_A -> /Pico/Motor_3_B
- U5 pad 9: /Pico/Motor_3_B -> /Pico/Motor_4_B
- U6 pad 10: /Pico/Motor_5_A -> /Pico/Motor_6_A
- U6 pad 12: VCC -> +3.3V
- U6 pad 2: /Pico/M5_Out_A -> /Pico/M6_Out_A
- U6 pad 3: /Pico/M5_Out_B -> /Pico/M6_Out_B
- U6 pad 4: /Pico/M6_Out_A -> /Pico/M5_Out_B
- U6 pad 5: /Pico/M6_Out_B -> /Pico/M5_Out_A
- U6 pad 7: /Pico/Motor_6_A -> /Pico/Motor_5_A
- U6 pad 8: /Pico/Motor_6_A -> /Pico/Motor_5_B
- U6 pad 9: /Pico/Motor_5_B -> /Pico/Motor_6_B
- U8 pad 10: /ESP_PICO_UART_TX -> /ESP32-S3-WROOM-1/GPIO_17
- U8 pad 11: /ESP_PICO_UART_RX -> /ESP32-S3-WROOM-1/GPIO_18
- U8 pad 12: unconnected-(U8-GPIO8/TOUCH8/ADC1_CH7/SUBSPICS1-Pad12) -> /ESP32-S3-WROOM-1/GPIO_8
- U8 pad 15: unconnected-(U8-GPIO3/TOUCH3/ADC1_CH2-Pad15) -> /ESP32-S3-WROOM-1/Battery_Voltage_Monitor
- U8 pad 2: Net-(U8-3V3) -> +3.3V
- U8 pad 26: /ESP32-S3-WROOM-1/LED_DIN -> unconnected-(U8-GPIO45-Pad26)
- U8 pad 3: Net-(U8-3V3) -> Net-(U8-EN)
- U8 pad 36: unconnected-(U8-U0RXD/GPIO44/CLK_OUT2-Pad36) -> /ESP_PICO_UART_RX
- U8 pad 37: unconnected-(U8-U0TXD/GPIO43/CLK_OUT1-Pad37) -> /ESP_PICO_UART_TX
- U8 pad 39: /ESP32-S3-WROOM-1/Battery_Voltage_Monitor -> /ESP32-S3-WROOM-1/LED_DIN
- U8 pad 8: unconnected-(U8-GPIO15/U0RTS/ADC2_CH4/XTAL_32K_P-Pad8) -> /ESP32-S3-WROOM-1/GPIO_15
- U8 pad 9: unconnected-(U8-GPIO16/U0CTS/ADC2_CH5/XTAL_32K_N-Pad9) -> /ESP32-S3-WROOM-1/GPIO_16
Routing:
- net /ESP_USB_D+: track 0.00 -> 28.2 mm
- net /ESP_USB_D-: track 0.00 -> 27.6 mm
- net /ESP32-S3-WROOM-1/LED_DIN: track 0.00 -> 25.4 mm
- net VCC: track 0.00 -> 22.0 mm
- net Earth: track 5.38 -> 24.0 mm, vias 2 -> 9
- net /ESP32-S3-WROOM-1/GPIO_8: track 0.00 -> 14.4 mm
- net /ESP32-S3-WROOM-1/GPIO_18: track 0.00 -> 13.5 mm
- net /ESP32-S3-WROOM-1/GPIO_17: track 0.00 -> 12.9 mm
- net Net-(Q3-G): track 0.00 -> 12.8 mm
- net /ESP32-S3-WROOM-1/ESP32CAM/ESPCAM_USB_D-: track 0.00 -> 12.7 mm
- net /ESP32-S3-WROOM-1/GPIO_16: track 0.00 -> 12.4 mm
- net /ESP32-S3-WROOM-1/GPIO_15: track 0.00 -> 11.9 mm
- net /ESP32-S3-WROOM-1/ADC0: track 0.00 -> 11.6 mm
- net /ESP32-S3-WROOM-1/ADC3: track 0.00 -> 11.4 mm
- net /ESP32-S3-WROOM-1/ADC1: track 0.00 -> 11.1 mm
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Other:
- board size 76.2 x 76.2 mm -> 75 x 75 mm

Commit message: Much much more progress
Parts:
- removed D1: SS34, Diode_SMD:D_SOD-123
- removed J10: Conn_01x02, Connector_JST:JST_XH_B2B-XH-AM_1x02_P2.50mm_Vertical
- removed J8, J9: Conn_01x08, Connector_PinSocket_2.54mm:PinSocket_1x08_P2.54mm_Vertical
- removed Q4: DMN65D8L, Package_TO_SOT_SMD:SOT-23
- removed R11: 220, Resistor_SMD:R_0402_1005Metric
- removed R19: 10k, Resistor_SMD:R_0402_1005Metric
- removed SW6: SW_Push, Button_Switch_SMD:SW_SPST_PTS645
- removed U9: AMS1117-1.8, Package_TO_SOT_SMD:SOT-223-3_TabPin2
- added C28: 0.1uF, Capacitor_SMD:C_0402_1005Metric, F.Cu at (231.9, 55.0)
- added C29: 0.1uF, Capacitor_SMD:C_0402_1005Metric, F.Cu at (161.9, 125.2)
- added C30: 1uF, Capacitor_SMD:C_0201_0603Metric, F.Cu at (181.9, 96.9)
- added C31: 1uF, Capacitor_SMD:C_0201_0603Metric, F.Cu at (188.2, 95.7)
- added C32: 100nF, Capacitor_SMD:C_0402_1005Metric, F.Cu at (211.0, 69.2)
- added C33: 100nF, Capacitor_SMD:C_0402_1005Metric, F.Cu at (217.1, 137.4)
- added C34: .1uf, Capacitor_SMD:C_0402_1005Metric, F.Cu at (178.2, 129.4)
- added C5: .1uF, Capacitor_SMD:C_0402_1005Metric, F.Cu at (205.1, 36.0)
- added J14: Conn_01x09, Connector_PinSocket_2.54mm:PinSocket_1x09_P2.54mm_Vertical, F.Cu at (201.8, 55.2)
- added J15: Conn_02x09_Top_Bottom, Connector_PinSocket_2.54mm:PinSocket_2x09_P2.54mm_Vertical, F.Cu at (207.0, 55.2)
- added J5: B4B-ZRLFSN, JST-ZR-4Pin:CONN_B4B-ZRLFSN_JST, F.Cu at (213.0, 114.0)
- added Q5: BSS138, Package_TO_SOT_SMD:SOT-23, F.Cu at (196.5, 113.2)
- added R14: 1K, Resistor_SMD:R_0402_1005Metric, F.Cu at (159.0, 68.5)
- added R33: 2.2k, Resistor_SMD:R_0402_1005Metric, F.Cu at (193.4, 112.8)
- added R34: 2.2k, Resistor_SMD:R_0402_1005Metric, F.Cu at (199.5, 112.6)
- added U13: MIC5365-3.3YC5, Package_TO_SOT_SMD:SOT-353_SC-70-5, F.Cu at (185.8, 96.8)
- C2: footprint Capacitor_SMD:C_0402_1005Metric -> Capacitor_SMD:C_Elec_6.3x5.8
- J11: value Conn_01x07 -> Conn_01x08; footprint Connector_PinSocket_2.54mm:PinSocket_1x07_P2.54mm_Vertical -> Connector_PinSocket_2.54mm:PinSocket_1x08_P2.54mm_Vertical
- J4: value Conn_01x02 -> B4B-ZRLFSN; footprint Connector_PinHeader_2.54mm:PinHeader_1x02_P2.54mm_Vertical -> JST-ZR-4Pin:CONN_B4B-ZRLFSN_JST
- Q2: value DMN65D8L -> BSS138
- R13: renamed from R14; footprint Resistor_SMD:R_0612_1632Metric -> Resistor_SMD:R_0402_1005Metric
- R18: footprint Resistor_SMD:R_0612_1632Metric -> Resistor_SMD:R_0402_1005Metric
- moved J12 171.2 mm to (152.3, 111.6), turned to -90 degrees
- moved C27 170.6 mm to (160.6, 118.6), turned to 180 degrees
- moved R29 168.8 mm to (162.4, 118.6), turned to 0 degrees
- moved C26 167.6 mm to (161.1, 116.3), turned to 90 degrees
- moved U12 166.9 mm to (160.9, 111.2), turned to 90 degrees
- moved R30 166.5 mm to (162.4, 116.3), turned to -90 degrees
- moved R18 164.7 mm to (183.3, 130.4)
- moved R20 162.6 mm to (204.0, 88.0), turned to 90 degrees
- moved R25 162.4 mm to (169.6, 118.3), turned to -90 degrees
- moved R31 161.9 mm to (154.6, 95.9), turned to 90 degrees
- moved C13 158.4 mm to (180.5, 118.2), turned to 180 degrees
- moved U11 158.2 mm to (165.7, 111.5), turned to -90 degrees
- moved C14 151.4 mm to (180.5, 116.9), turned to 180 degrees
- moved R10 148.0 mm to (208.8, 108.9), turned to 90 degrees
- moved R28 146.9 mm to (171.4, 118.3), turned to 90 degrees
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- renumbered SW3 to Boot1, C5 to C4, SW2 to RST1, J5 to SWD1
Connections:
- net /ESP32-S3-WROOM-1/ESP32CAM/USB_RX renamed /ESP32-S3-WROOM-1/USB_TX
- net /ESP32-S3-WROOM-1/ESP32CAM/USB_TX renamed /ESP32-S3-WROOM-1/USB_RX
- C3 pad 1: Net-(Q3-S) -> VCC
- C4 pad 1: Net-(C5-Pad1) -> +3.3V
- D2 pad 3: Net-(Q3-S) -> VCC
- J1 pad 2: VCC -> VS
- J11 pad 2: /ESP32-S3-WROOM-1/ESP_MISO -> /ESP32-S3-WROOM-1/Handshake2
- J11 pad 3: /ESP32-S3-WROOM-1/ESP_SCLK -> /ESP32-S3-WROOM-1/ESP_MISO
- J11 pad 4: /ESP32-S3-WROOM-1/ESP_MOSI -> /ESP32-S3-WROOM-1/ESP_SCLK
- J11 pad 5: /ESP32-S3-WROOM-1/ESP_CS0 -> /ESP32-S3-WROOM-1/ESP_MOSI
- J11 pad 6: +3.3V -> /ESP32-S3-WROOM-1/ESP_CS0
- J11 pad 7: +5V -> +3.3V
- J4 pad 1: /Pico/I2C_SDA -> +3.3V
- J4 pad 2: /Pico/I2C_SCL -> /ESP32-S3-WROOM-1/SDA
- J7 pad 19: unconnected-(J7-Pin_19-Pad19) -> /ESP32-S3-WROOM-1/ESP_MISO
- J7 pad 2: unconnected-(J7-Pin_2-Pad2) -> +5V
- J7 pad 20: Earth -> unconnected-(J7-Pin_20-Pad20)
- J7 pad 21: unconnected-(J7-Pin_21-Pad21) -> /ESP32-S3-WROOM-1/ESP_MOSI
- J7 pad 23: unconnected-(J7-Pin_23-Pad23) -> /ESP32-S3-WROOM-1/ESP_SCLK
- J7 pad 24: unconnected-(J7-Pin_24-Pad24) -> /ESP32-S3-WROOM-1/ESP_CS1
- J7 pad 25: unconnected-(J7-Pin_25-Pad25) -> Earth
- J7 pad 38: Earth -> unconnected-(J7-Pin_38-Pad38)
- J7 pad 39: unconnected-(J7-Pin_39-Pad39) -> Earth
- J7 pad 4: unconnected-(J7-Pin_4-Pad4) -> +5V
- J7 pad 40: +5V -> unconnected-(J7-Pin_40-Pad40)
- J7 pad 6: unconnected-(J7-Pin_6-Pad6) -> Earth
- J7 pad 9: unconnected-(J7-Pin_9-Pad9) -> Earth
- Q1 pad 3: Net-(Q1B-C2) -> Net-(Q1A-C1)
- Q2 pad 2: /Pico/I2C_SDA -> /Pico/IMU/SDA
- Q2 pad 3: /Pico/IMU/SDA -> /Pico/I2C_SDA
- Q3 pad 2: VCC -> VS
- Q3 pad 3: Net-(Q3-S) -> VCC
- R10 pad 2: Net-(Q1B-C2) -> Net-(Q1A-C1)
- R12 pad 1: /ESP_PICO_UART_TX -> ESP_TX
- R13 pad 1: Net-(U4-RUN) -> ESP_RX
- R13 pad 2: +3.3V -> Net-(Q1A-B1)
- R13 pad 1: /ESP_PICO_UART_RX -> ESP_RX
- R22 pad 2: /Pico/I2C_SDA -> /Pico/IMU/SDA
- R23 pad 2: /Pico/IMU/SDA -> /Pico/I2C_SDA
- R29 pad 2: Net-(U11-USBDM) -> /ESP32-S3-WROOM-1/ESP32CAM/3.3V_Out
- R30 pad 1: Net-(U11-USBDP) -> /ESP32-S3-WROOM-1/ESP32CAM/3.3V_Out
- R32 pad 1: VCC -> VS
- RST1 pad 1: +3.3V -> /ESP_PU
- SW5 pad 2: Earth -> unconnected-(SW5-Pad2)
- U1 pad 2: Net-(Q3-S) -> VCC
- U1 pad 3: Net-(Q3-S) -> VCC
- U10 pad 23: /Pico/I2C_SCL -> /Pico/IMU/SCL
- U10 pad 24: /Pico/I2C_SDA -> /Pico/IMU/SDA
- U11 pad 11: Net-(U11-USBDP) -> /ESP32-S3-WROOM-1/ESP32CAM/3.3V_Out
- U11 pad 12: Net-(U11-USBDM) -> /ESP32-S3-WROOM-1/ESP32CAM/3.3V_Out
- U12 pad P$11: /ESP32-S3-WROOM-1/ESP_MOSI -> /ESP32-S3-WROOM-1/ESP_MISO
- U12 pad P$12: /ESP32-S3-WROOM-1/ESP_MISO -> /ESP32-S3-WROOM-1/ESP_MOSI
- U12 pad P$13: /ESP32-S3-WROOM-1/ESP_CS2 -> /ESP32-S3-WROOM-1/ESP_CS1
- U2 pad 3: Net-(Q3-S) -> VCC
- U4 pad 15: unconnected-(U4-GPIO12-Pad15) -> ESP_RX
- U4 pad 16: /ESP_PICO_UART_RX -> ESP_TX
- U4 pad 17: /ESP_PICO_UART_TX -> unconnected-(U4-GPIO14-Pad17)
- U4 pad 26: Net-(U4-RUN) -> /ESP_PU
- U4 pad 29: /Pico/M1_Enc_A -> /Pico/M1_Enc_B
- U4 pad 30: /Pico/M1_Enc_B -> /Pico/M1_Enc_A
- U8 pad 16: /ESP32-S3-WROOM-1/ESP_CS2 -> /ESP32-S3-WROOM-1/Handshake
- U8 pad 22: /ESP32-S3-WROOM-1/Handshake -> /ESP32-S3-WROOM-1/Handshake2
- U8 pad 23: unconnected-(U8-GPIO21-Pad23) -> /ESP32-S3-WROOM-1/ESP_CS2
- U8 pad 26: unconnected-(U8-GPIO45-Pad26) -> /ESP32-S3-WROOM-1/GPIO45
- U8 pad 28: unconnected-(U8-SPIIO6/GPIO35/FSPID/SUBSPID-Pad28) -> /ESP32-S3-WROOM-1/GPIO35
- U8 pad 29: unconnected-(U8-SPIIO7/GPIO36/FSPICLK/SUBSPICLK-Pad29) -> /ESP32-S3-WROOM-1/GPIO36
- U8 pad 3: Net-(U8-EN) -> /ESP_PU
- U8 pad 30: unconnected-(U8-SPIDQS/GPIO37/FSPIQ/SUBSPIQ-Pad30) -> /ESP32-S3-WROOM-1/GPIO37
- U8 pad 31: unconnected-(U8-GPIO38/FSPIWP/SUBSPIWP-Pad31) -> /ESP32-S3-WROOM-1/GPIO38
- U8 pad 32: unconnected-(U8-MTCK/GPIO39/CLK_OUT3/SUBSPICS1-Pad32) -> /ESP32-S3-WROOM-1/GPIO39
- U8 pad 33: unconnected-(U8-MTDO/GPIO40/CLK_OUT2-Pad33) -> /ESP32-S3-WROOM-1/GPIO40
- U8 pad 34: unconnected-(U8-MTDI/GPIO41/CLK_OUT1-Pad34) -> /ESP32-S3-WROOM-1/GPIO41
- U8 pad 35: unconnected-(U8-MTMS/GPIO42-Pad35) -> /ESP32-S3-WROOM-1/GPIO42
- U8 pad 36: /ESP_PICO_UART_RX -> ESP_RX
- U8 pad 37: /ESP_PICO_UART_TX -> ESP_TX
Routing:
- net +3.3V: track 7.03 -> 276.6 mm, vias 1 -> 13
- net Earth: track 24.0 -> 258.5 mm, vias 9 -> 43
- net VCC: track 22.0 -> 142.5 mm, vias 0 -> 9
- net ESP_TX: track 0.00 -> 81.4 mm, vias 0 -> 3
- net ESP_RX: track 0.00 -> 80.4 mm, vias 0 -> 3
- net +5V: track 0.00 -> 60.6 mm, vias 0 -> 3
- net Net-(U4-USB_DM): track 0.00 -> 53.0 mm
- net Net-(U4-USB_DP): track 0.00 -> 52.6 mm
- net /ESP32-S3-WROOM-1/ESP_SCLK: track 0.00 -> 50.5 mm, vias 0 -> 1
- net /ESP32-S3-WROOM-1/Handshake: track 0.00 -> 48.2 mm, vias 0 -> 1
- net /ESP32-S3-WROOM-1/ESP_MISO: track 0.00 -> 45.8 mm, vias 0 -> 1
- net /ESP32-S3-WROOM-1/ESP_CS1: track 0.00 -> 44.7 mm, vias 0 -> 1
- net /ESP32-S3-WROOM-1/ESP_MOSI: track 0.00 -> 43.8 mm, vias 0 -> 1
- net /ESP_PU: track 0.00 -> 37.2 mm, vias 0 -> 3
- net Net-(Boot1-Pad1): track 0.00 -> 36.0 mm, vias 0 -> 2
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Other:
- board size 75 x 75 mm -> 75 x 100 mm
- board text added: "Batt"
- board text added: "Status"

Commit message: Rev 1
Parts:
- removed the C28 at (231.9, 55.0)
- removed C29 (x2): 0.1uF, Capacitor_SMD:C_0402_1005Metric
- removed the C4 at (75.0, 78.3)
- removed the R13 at (41.6, 37.8)
- removed R17: DNF, Resistor_SMD:R_0612_1632Metric
- removed R3, R31, R9: 1M, Resistor_SMD:R_0402_1005Metric
- removed SW5: SW_Push, Button_Switch_SMD:SW_SPST_PTS645
- added C35: 1uf, Capacitor_SMD:C_0201_0603Metric, F.Cu at (193.4, 121.7)
- added C36: 100nF, Capacitor_SMD:C_0201_0603Metric, F.Cu at (199.8, 129.3)
- added C37: 100nF, Capacitor_SMD:C_0201_0603Metric, F.Cu at (206.4, 123.2)
- added C38: 100nF, Capacitor_SMD:C_0201_0603Metric, F.Cu at (199.6, 117.6)
- added C39: 100nF, Capacitor_SMD:C_0201_0603Metric, F.Cu at (195.0, 118.9)
- added C40: 100nF, Capacitor_SMD:C_0201_0603Metric, F.Cu at (192.5, 123.4)
- added C41: 1uf, Capacitor_SMD:C_0201_0603Metric, F.Cu at (193.7, 120.6)
- added C42: 100nF, Capacitor_SMD:C_0201_0603Metric, F.Cu at (192.8, 124.1)
- added J10: Conn_01x02, Connector_PinHeader_2.54mm:PinHeader_1x02_P2.54mm_Vertical, F.Cu at (163.5, 127.6)
- C10, C7, C8, C9: footprint Capacitor_SMD:C_0402_1005Metric -> Capacitor_SMD:C_0201_0603Metric
- C3: footprint Capacitor_SMD:C_0402_1005Metric -> Capacitor_SMD:C_0805_2012Metric
- moved C18 175.1 mm to (213.9, 72.8), turned to 180 degrees
- moved C7 168.2 mm to (193.7, 119.8), turned to 180 degrees
- moved C8 167.6 mm to (192.9, 117.9)
- moved C17 134.6 mm to (172.0, 51.7), turned to -90 degrees
- moved C3 101.0 mm to (168.5, 90.2), turned to 180 degrees
- moved R1 97.5 mm to (160.1, 76.8)
- moved R2 97.2 mm to (159.5, 72.4), turned to 90 degrees
- moved C28 88.2 mm to (165.5, 117.9), turned to 0 degrees
- moved R27 57.4 mm to (153.8, 104.5), turned to 90 degrees
- moved R26 56.1 mm to (152.8, 104.4), turned to 90 degrees
- moved C5 54.9 mm to (159.5, 66.7)
- moved C4 51.6 mm to (166.7, 80.8)
- moved C25 48.5 mm to (157.3, 118.1), turned to -90 degrees
- moved SW4 41.1 mm to (213.9, 76.3)
- moved C10 40.8 mm to (205.2, 122.6), turned to 0 degrees
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Connections:
- C10 pad 1: +3.3V -> Net-(U4-VREG_VOUT)
- C10 pad 2: Net-(C10-Pad2) -> Earth
- C7 pad 2: Net-(U4-VREG_IN) -> Earth
- C8 pad 2: Net-(U4-USB_VDD) -> Earth
- C9 pad 1: +3.3V -> Earth
- C9 pad 2: Net-(C9-Pad2) -> +3.3V
- J12 pad S1: Net-(J12-SHIELD) -> Earth
- J2 pad S1: Net-(J2-SHIELD) -> Earth
- J3 pad S1: Net-(J3-SHIELD) -> Earth
- J4 pad 1: +3.3V -> +5V
- J5 pad 1: +3.3V -> +5V
- R29 pad 2: /ESP32-S3-WROOM-1/ESP32CAM/3.3V_Out -> Net-(U11-USBDM)
- R30 pad 1: /ESP32-S3-WROOM-1/ESP32CAM/3.3V_Out -> Net-(U11-USBDP)
- U11 pad 11: /ESP32-S3-WROOM-1/ESP32CAM/3.3V_Out -> Net-(U11-USBDP)
- U11 pad 12: /ESP32-S3-WROOM-1/ESP32CAM/3.3V_Out -> Net-(U11-USBDM)
- U4 pad 1: Net-(C9-Pad2) -> +3.3V
- U4 pad 10: Net-(C9-Pad2) -> +3.3V
- U4 pad 22: Net-(C9-Pad2) -> +3.3V
- U4 pad 23: Net-(C10-Pad2) -> Net-(U4-VREG_VOUT)
- U4 pad 33: Net-(C9-Pad2) -> +3.3V
- U4 pad 42: Net-(C9-Pad2) -> +3.3V
- U4 pad 43: unconnected-(U4-ADC_AVDD-Pad43) -> +3.3V
- U4 pad 44: Net-(U4-VREG_IN) -> +3.3V
- U4 pad 45: Earth -> Net-(U4-VREG_VOUT)
- U4 pad 48: Net-(U4-USB_VDD) -> +3.3V
- U4 pad 49: Net-(C9-Pad2) -> +3.3V
- U4 pad 50: Net-(C10-Pad2) -> Net-(U4-VREG_VOUT)
Routing:
- net /ESP_PU: track 37.2 -> 161.1 mm, vias 3 -> 4
- net +3.3V: track 276.6 -> 372.1 mm, vias 13 -> 17
- net Earth: track 258.5 -> 327.3 mm, vias 43 -> 54
- net +5V: track 60.6 -> 105.7 mm
- net Net-(U8-GPIO0/BOOT): track 0.00 -> 25.8 mm
- net +1V8: track 19.1 -> 42.2 mm
- net Net-(U4-VREG_VOUT): track 0.00 -> 22.0 mm, vias 0 -> 3
- net /ESP32-S3-WROOM-1/ESP32CAM/V_USB: track 12.5 -> 24.0 mm, vias 2 -> 3
- net Net-(J12-CC2): track 0.00 -> 9.96 mm
- net VS: track 26.4 -> 16.5 mm
- net Net-(J12-CC1): track 0.00 -> 6.56 mm
- net Net-(J10-Pin_2): track 0.00 -> 5.44 mm
- net Net-(U11-USBDM): track 0.00 -> 4.73 mm
- net /Pico/USB_DP_Pico: track 0.00 -> 4.25 mm
- net /ESP32-S3-WROOM-1/ESP32CAM/3.3V_Out: track 6.55 -> 10.8 mm
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
Commit message: Rev0.1
Parts:
- removed C8: 100nF, Capacitor_SMD:C_0201_0603Metric
- removed REF** (x4): MountingHole_3.2mm_M3_ISO14580_Pad_TopOnly, MountingHole:MountingHole_3.2mm_M3_ISO14580_Pad_TopOnly
- added H1: MountingHole_Pad, MountingHole:MountingHole_3.2mm_M3_ISO14580_Pad_TopOnly, F.Cu at (155.0, 55.0)
- added H2: MountingHole_Pad, MountingHole:MountingHole_3.2mm_M3_ISO14580_Pad_TopOnly, F.Cu at (220.0, 55.0)
- added H3: MountingHole_Pad, MountingHole:MountingHole_3.2mm_M3_ISO14580_Pad_TopOnly, F.Cu at (155.0, 145.0)
- added H4: MountingHole_Pad, MountingHole:MountingHole_3.2mm_M3_ISO14580_Pad_TopOnly, F.Cu at (220.0, 145.0)
- added TP1: TestPoint_2Pole, TestPoint:TestPoint_2Pads_Pitch2.54mm_Drill0.8mm, F.Cu at (204.2, 105.3)
- moved R16 46.4 mm to (190.4, 121.2)
- moved R15 46.4 mm to (190.4, 122.2)
- moved R12 3.43 mm to (207.8, 103.8)
- moved R13 2.46 mm to (207.8, 106.1)
- moved R10 2.03 mm to (210.9, 108.7)
- moved D3 2.03 mm to (209.6, 108.7)
- moved D4 2.03 mm to (212.1, 108.7)
- moved Q1 2.03 mm to (210.7, 105.9)
- moved J1 1.72 mm to (154.9, 129.7)
- moved C34 1.29 mm to (179.0, 130.4)
- moved C38 0.94 mm to (200.3, 116.9), turned to -90 degrees
- moved C17 0.41 mm to (171.6, 51.6)
- moved J13 0.25 mm to (165.3, 52.9)
- moved R6 0.17 mm to (162.8, 86.2)
- moved C16 0.14 mm to (172.9, 51.6)
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Connections:
- J5 pad 2: /Pico/I2C_SDA -> PICO_SDA
- J5 pad 3: /Pico/I2C_SCL -> PICO_SCL
- J7 pad 19: /ESP32-S3-WROOM-1/ESP_MISO -> unconnected-(J7-Pin_19-Pad19)
- J7 pad 21: /ESP32-S3-WROOM-1/ESP_MOSI -> unconnected-(J7-Pin_21-Pad21)
- J7 pad 23: /ESP32-S3-WROOM-1/ESP_SCLK -> unconnected-(J7-Pin_23-Pad23)
- J7 pad 24: /ESP32-S3-WROOM-1/ESP_CS1 -> unconnected-(J7-Pin_24-Pad24)
- J7 pad 27: unconnected-(J7-Pin_27-Pad27) -> /ESP32-S3-WROOM-1/SDA
- J7 pad 28: unconnected-(J7-Pin_28-Pad28) -> /ESP32-S3-WROOM-1/SCL
- J7 pad 3: unconnected-(J7-Pin_3-Pad3) -> PICO_SDA
- J7 pad 5: unconnected-(J7-Pin_5-Pad5) -> PICO_SCL
- Q2 pad 3: /Pico/I2C_SDA -> PICO_SDA
- Q5 pad 3: /Pico/I2C_SCL -> PICO_SCL
- R23 pad 2: /Pico/I2C_SDA -> PICO_SDA
- R34 pad 2: /Pico/I2C_SCL -> PICO_SCL
- U12 pad P$11: /ESP32-S3-WROOM-1/ESP_MISO -> /ESP32-S3-WROOM-1/ESP_MOSI
- U12 pad P$12: /ESP32-S3-WROOM-1/ESP_MOSI -> /ESP32-S3-WROOM-1/ESP_MISO
- U4 pad 27: /Pico/I2C_SDA -> PICO_SDA
- U4 pad 28: /Pico/I2C_SCL -> PICO_SCL
Routing:
- net +3.3V: track 372.1 -> 85.7 mm, vias 17 -> 18
- net Earth: track 327.3 -> 234.8 mm, vias 54 -> 50
- net /Pico/USB_DP_Pico: track 4.25 -> 53.7 mm
- net /Pico/USB_DM_Pico: track 2.21 -> 51.3 mm
- net Net-(U4-USB_DM): track 53.8 -> 4.84 mm
- net Net-(U4-USB_DP): track 53.4 -> 4.60 mm
- net PICO_SCL: track 0.00 -> 43.2 mm, vias 0 -> 1
- net PICO_SDA: track 0.00 -> 41.2 mm
- net +5V: track 105.7 -> 136.8 mm
- net /Pico/I2C_SDA: track 27.0 -> 0.00 mm
- net /Pico/I2C_SCL: track 25.9 -> 0.00 mm, vias 1 -> 0
- net /ESP32-S3-WROOM-1/SDA: track 23.3 -> 45.2 mm
- net /ESP32-S3-WROOM-1/SCL: track 23.4 -> 40.8 mm
- net VS: track 16.5 -> 10.4 mm
- net /ESP_PU: track 161.1 -> 165.8 mm
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- added copper zone on In2.Cu, net +3.3V
- added copper zone on In1.Cu, net Earth
Other:
- board text added: "WPI SRL Rev 1.0.0 Designed by: Nikesh Walling Date: 2/2/2024"

Commit message: clean up Rev
Parts:
- C3: footprint Capacitor_SMD:C_0805_2012Metric -> Capacitor_SMD:C_0402_1005Metric
- C34: footprint Capacitor_SMD:C_0402_1005Metric -> Capacitor_SMD:C_0805_2012Metric
- moved C19 0.24 mm to (171.8, 55.1)
Routing:
- net Earth: track 234.8 -> 233.4 mm
- net /Pico/M2_Enc_A: track 28.6 -> 27.7 mm
- net /Pico/M1_Enc_B: track 34.4 -> 33.7 mm
- net /Pico/M4_Enc_A: track 32.6 -> 31.9 mm
Other:
- board text added: "WPI SRL Rev 1.0.0 Designer : Nikesh Walling Date: 2/12/2024"
- board text removed: "WPI SRL Rev 1.0.0 Designed by: Nikesh Walling Date: 2/2/2024"
