File: ESP32-S3-WROOM-1.kicad_sch (KiCad schematic)
At the start: 7 parts, among them SW3 SW_Push, U8 ESP32-S3-WROOM-1

Commit message: More progress
Parts:
- removed R23: 10k, symbol Device:R_US
- added C16: 1uf, Capacitor_SMD:C_0402_1005Metric, symbol Device:C_Small
- added C17, C19, C20, C21: 0.1uF, Capacitor_SMD:C_0402_1005Metric, symbol Device:C_Small
- added D6: WS2812B, LED_SMD:LED_WS2812B_PLCC4_5.0x5.0mm_P3.2mm, symbol LED:WS2812B
- added J10: Conn_01x02, Connector_JST:JST_XH_B2B-XH-AM_1x02_P2.50mm_Vertical, symbol Connector_Generic:Conn_01x02
- added J11: Conn_01x07, Connector_PinSocket_2.54mm:PinSocket_1x07_P2.54mm_Vertical, symbol Connector_Generic:Conn_01x07
- added J6: Conn_02x20_Counter_Clockwise, Connector_PinSocket_2.54mm:PinSocket_2x20_P2.54mm_Vertical, symbol Connector_Generic:Conn_02x20_Counter_Clockwise
- added J7, J8: Conn_01x08, Connector_PinSocket_2.54mm:PinSocket_1x08_P2.54mm_Vertical, symbol Connector_Generic:Conn_01x08
- added J9: Conn_01x04, Connector_PinSocket_2.54mm:PinSocket_1x04_P2.54mm_Vertical, symbol Connector_Generic:Conn_01x04
- added R19: 10k, Resistor_SMD:R_0402_1005Metric, symbol Device:R_US
- added R20, R21: 5k, Resistor_SMD:R_0402_1005Metric, symbol Device:R_Small_US
- added SW5: SW_Push, Button_Switch_SMD:SW_SPST_PTS645, symbol Switch:SW_Push
- C14: renamed from C17; value 22uF -> 22uf; footprint (none) -> Capacitor_SMD:C_0402_1005Metric
- C15: renamed from C16; footprint (none) -> Capacitor_SMD:C_0402_1005Metric
- C18: footprint (none) -> Capacitor_SMD:C_0402_1005Metric
- SW4: renamed from SW3; footprint (none) -> Button_Switch_SMD:SW_SPST_PTS645
- U8: value ESP32-S3-WROOM-1 -> ESP32-S3-WROOM-1-N8R2; footprint PCM_Espressif:ESP32-S3-WROOM-1 -> Espressif:ESP32-S3-WROOM-1
- renumbered D5 to D7
Connections:
- net +3.3V: now also J11.6 (Pin_6), J7.8 (Pin_8), R19.2, R20.1, R21.1; no longer U8.2 (3V3)
- net Earth: now also C18.1, C16.1, C17.1, C19.1, C20.1, C21.1, D6.3 (VSS), J11.1 (Pin_1), J6.20 (Pin_20), J6.38 (Pin_38), J7.1 (Pin_1), J7.5 (Pin_5), J8.7 (Pin_7), SW5.2; no longer C18.2
- net at C15.2, SW4.2, U8.3 (EN): now also C14.1, U8.2 (3V3), C16.2, R19.1
- net +5V: now reaches D7.1 (VDD)
- net +5V: now also D6.1 (VDD), J11.7 (Pin_7), J6.40 (Pin_40)
- net at D7.2 (DOUT): now also D6.4 (DIN)
- net LED_DIN: now reaches D7.4 (DIN)
- net LED_DIN: now also U8.26 (GPIO45)
- net ESP_UART_TX: now reaches U8.10 (GPIO17/U1TXD/ADC2_CH6)
- net ESP_UART_RX: now reaches U8.11 (GPIO18/U1RXD/ADC2_CH7/CLK_OUT3)
- net USB_D-: now reaches U8.13 (GPIO19/U1RTS/ADC2_CH8/CLK_OUT2/USB_D-)
- net USB_D+: now reaches U8.14 (GPIO20/U1CTS/ADC2_CH9/CLK_OUT1/USB_D+)
- net ESP_CS2: now reaches U8.16 (GPIO46)
- net ESP_CS1: now reaches U8.17 (GPIO9/TOUCH9/ADC1_CH8/FSPIHD/SUBSPIHD)
- net ESP_CS0: now reaches U8.18 (GPIO10/TOUCH10/ADC1_CH9/FSPICS0/FSPIIO4/SUBSPICS0)
- net ESP_CS0: now also J11.5 (Pin_5), J8.4 (Pin_4)
- net ESP_MOSI: now reaches U8.19 (GPIO11/TOUCH11/ADC2_CH0/FSPID/FSPIIO5/SUBSPID)
- net ESP_MOSI: now also J11.4 (Pin_4), J8.5 (Pin_5)
- net ESP_SCLK: now reaches U8.20 (GPIO12/TOUCH12/ADC2_CH1/FSPICLK/FSPIIO6/SUBSPICLK)
- net ESP_SCLK: now also J11.3 (Pin_3), J8.3 (Pin_3)
- net ESP_MISO: now reaches U8.21 (GPIO13/TOUCH13/ADC2_CH2/FSPIQ/FSPIIO7/SUBSPIQ)
- net ESP_MISO: now also J11.2 (Pin_2), J8.6 (Pin_6)
- net Handshake: now reaches U8.22 (GPIO14/TOUCH14/ADC2_CH3/FSPIWP/FSPIDQS/SUBSPIWP)
- net Handshake: now also J8.2 (Pin_2)
- net SDA: now reaches U8.24 (GPIO47/SPICLK_P/SUBSPICLK_P_DIFF)
- net SDA: now also J10.1 (Pin_1), R20.2
- net SCL: now reaches U8.25 (GPIO48/SPICLK_N/SUBSPICLK_N_DIFF)
- net SCL: now also J10.2 (Pin_2), R21.2
- net Battery_Voltage_Monitor: now reaches U8.39 (GPIO1/TOUCH1/ADC1_CH0)
- net ADC0: now reaches U8.4 (GPIO4/TOUCH4/ADC1_CH3)
- net ADC0: now also C21.2, J9.4 (Pin_4)
- net ADC1: now reaches U8.5 (GPIO5/TOUCH5/ADC1_CH4)
- net ADC1: now also C20.2, J9.3 (Pin_3)
- net ADC2: now reaches U8.6 (GPIO6/TOUCH6/ADC1_CH5)
- net ADC2: now also C19.2, J9.2 (Pin_2)
- net ADC3: now reaches U8.7 (GPIO7/TOUCH7/ADC1_CH6)
- net ADC3: now also C18.2, J9.1 (Pin_1)
- net PIO_0_Boot: no longer names the net of U8.27 (GPIO0/BOOT)
- net PIO_0_Boot: now also C17.2, SW5.1
- no-connect marks 0 -> 8
Other:
- added sheet ESP32CAM (ESP32CAM.kicad_sch)
- note added: "ADC Ports"
- note added: "Battery Status"
- note added: "ESP CAM Port"
- note added: "ESP32-CAM"
- note added: "General Status"
- note added: "I2C Access"
- note added: "Raspberry Pi Interface"
- note added: "Spare SPI Port"
- note added: "Status LEDs"
- moved on the sheet: C14, C15, D7, SW4, U8

Commit message: Nearly done schematics
Parts:
- removed C14: 22uf, Capacitor_SMD:C_0402_1005Metric, symbol Device:C_Small
- removed C18: 0.1uF, Capacitor_SMD:C_0402_1005Metric, symbol Device:C_Small
- removed J9: Conn_01x04, Connector_PinSocket_2.54mm:PinSocket_1x04_P2.54mm_Vertical, symbol Connector_Generic:Conn_01x04
- removed R19: 10k, Resistor_SMD:R_0402_1005Metric, symbol Device:R_US
- removed SW4: SW_Push, Button_Switch_SMD:SW_SPST_PTS645, symbol Switch:SW_Push
- added C17: 22uf, Capacitor_SMD:C_0402_1005Metric, symbol Device:C_Small
- added C22: 0.1uF, Capacitor_SMD:C_0402_1005Metric, symbol Device:C_Small
- added J13: Conn_02x09_Top_Bottom, Connector_PinSocket_2.54mm:PinSocket_2x09_P2.54mm_Vertical, symbol Connector_Generic:Conn_02x09_Odd_Even
- added J6: Conn_01x09, Connector_PinSocket_2.54mm:PinSocket_1x09_P2.54mm_Vertical, symbol Connector_Generic:Conn_01x09
- SW4: renamed from SW5; footprint Button_Switch_SMD:SW_SPST_PTS645 -> Button_Switch_SMD:SW_SPST_PTS810
- renumbered C17 to C18, J6 to J7, J7 to J8, J8 to J9
Connections:
- net +3.3V: now also C15.2, C16.2, U8.2 (3V3), C17.2, J13.1 (Pin_1), J13.11 (Pin_11), J13.13 (Pin_13), J13.15 (Pin_15), J13.17 (Pin_17), J13.3 (Pin_3), J13.5 (Pin_5), J13.7 (Pin_7), J13.9 (Pin_9)
- net ADC0: now also C19.2, J6.1 (Pin_1); no longer C21.2
- net ADC1: now also J6.2 (Pin_2)
- net ADC2: now also C21.2, J6.3 (Pin_3); no longer C19.2
- net ADC3: now also C22.2, J6.4 (Pin_4)
- net Battery_Voltage_Monitor: now also U8.15 (GPIO3/TOUCH3/ADC1_CH2); no longer U8.39 (GPIO1/TOUCH1/ADC1_CH0)
- net ESP_UART_RX: now also U8.36 (U0RXD/GPIO44/CLK_OUT2); no longer U8.11 (GPIO18/U1RXD/ADC2_CH7/CLK_OUT3)
- net ESP_UART_TX: now also U8.37 (U0TXD/GPIO43/CLK_OUT1); no longer U8.10 (GPIO17/U1TXD/ADC2_CH6)
- net Earth: now also C17.1, C22.1, J13.10 (Pin_10), J13.12 (Pin_12), J13.14 (Pin_14), J13.16 (Pin_16), J13.18 (Pin_18), J13.2 (Pin_2), J13.4 (Pin_4), J13.6 (Pin_6), J13.8 (Pin_8)
- net LED_DIN: now also U8.39 (GPIO1/TOUCH1/ADC1_CH0); no longer U8.26 (GPIO45)
- net GPIO_8: now reaches U8.12 (GPIO8/TOUCH8/ADC1_CH7/SUBSPICS1)
- net GPIO_8: now also J6.9 (Pin_9)
- net GPIO_15: now reaches U8.8 (GPIO15/U0RTS/ADC2_CH4/XTAL_32K_P)
- net GPIO_15: now also J6.5 (Pin_5)
- net GPIO_16: now reaches U8.9 (GPIO16/U0CTS/ADC2_CH5/XTAL_32K_N)
- net GPIO_16: now also J6.6 (Pin_6)
- new net ESP_PU: U8.3 (EN)
- new net GPIO_17: J6.7 (Pin_7), U8.10 (GPIO17/U1TXD/ADC2_CH6)
- new net GPIO_18: J6.8 (Pin_8), U8.11 (GPIO18/U1RXD/ADC2_CH7/CLK_OUT3)
Other:
- note added: "Filtered ADC + GPIO Ports"
- note removed: "ADC Ports"
- moved on the sheet: C15, C16, J10, R20, R21

Commit message: Much much more progress
Parts:
- removed J10: Conn_01x02, Connector_JST:JST_XH_B2B-XH-AM_1x02_P2.50mm_Vertical, symbol Connector_Generic:Conn_01x02
- added C32: 100nF, Capacitor_SMD:C_0402_1005Metric, symbol Device:C_Small
- added J14: Conn_01x09, Connector_PinSocket_2.54mm:PinSocket_1x09_P2.54mm_Vertical, symbol Connector_Generic:Conn_01x09
- added J15: Conn_02x09_Top_Bottom, Connector_PinSocket_2.54mm:PinSocket_2x09_P2.54mm_Vertical, symbol Connector_Generic:Conn_02x09_Odd_Even
- added J4: B4B-ZRLFSN, JST-ZR-4Pin:CONN_B4B-ZRLFSN_JST, symbol JST-ZH-4Pin:B4B-ZRLFSN
- J11: value Conn_01x07 -> Conn_01x08; footprint Connector_PinSocket_2.54mm:PinSocket_1x07_P2.54mm_Vertical -> Connector_PinSocket_2.54mm:PinSocket_1x08_P2.54mm_Vertical; symbol Connector_Generic:Conn_01x07 -> Connector_Generic:Conn_01x08
- J7: symbol Connector_Generic:Conn_02x20_Counter_Clockwise -> Connector_Generic:Conn_02x20_Odd_Even; now in the parts list
- J8, J9: now not fitted
Connections:
- net +3.3V: now also J11.7 (Pin_7), J15.10 (Pin_10), J15.12 (Pin_12), J15.14 (Pin_14), J15.16 (Pin_16), J15.18 (Pin_18), J15.2 (Pin_2), J15.4 (Pin_4), J15.6 (Pin_6), J15.8 (Pin_8), J4.1; no longer J11.6 (Pin_6)
- net +5V: now also J7.2 (Pin_2), J7.4 (Pin_4), C32.2; no longer J11.7 (Pin_7), J7.40 (Pin_40)
- net ESP_CS0: now also J11.6 (Pin_6); no longer J11.5 (Pin_5)
- net ESP_CS1: now also J7.24 (Pin_24)
- net ESP_CS2: now also U8.23 (GPIO21); no longer U8.16 (GPIO46)
- net ESP_MISO: now also J11.3 (Pin_3), J7.19 (Pin_19); no longer J11.2 (Pin_2)
- net ESP_MOSI: now also J11.5 (Pin_5), J7.21 (Pin_21); no longer J11.4 (Pin_4)
- net ESP_SCLK: now also J11.4 (Pin_4), J7.23 (Pin_23); no longer J11.3 (Pin_3)
- net Earth: now also J7.25 (Pin_25), J7.39 (Pin_39), J7.6 (Pin_6), J7.9 (Pin_9), C32.1, J15.1 (Pin_1), J15.11 (Pin_11), J15.13 (Pin_13), J15.15 (Pin_15), J15.17 (Pin_17), J15.3 (Pin_3), J15.5 (Pin_5), J15.7 (Pin_7), J15.9 (Pin_9), J4.4; no longer J7.20 (Pin_20), J7.38 (Pin_38)
- net Handshake: now also U8.16 (GPIO46); no longer U8.22 (GPIO14/TOUCH14/ADC2_CH3/FSPIWP/FSPIDQS/SUBSPIWP)
- net SCL: now also J4.3
- net SDA: now also J4.2
- net USB_RX: now reaches J8.2 (Pin_2)
- net USB_TX: now reaches J8.3 (Pin_3)
- net GPIO45: now reaches U8.26 (GPIO45)
- net GPIO45: now also J14.9 (Pin_9)
- net GPIO35: now reaches U8.28 (SPIIO6/GPIO35/FSPID/SUBSPID)
- net GPIO35: now also J14.8 (Pin_8)
- net GPIO36: now reaches U8.29 (SPIIO7/GPIO36/FSPICLK/SUBSPICLK)
- net GPIO36: now also J14.7 (Pin_7)
- net GPIO37: now reaches U8.30 (SPIDQS/GPIO37/FSPIQ/SUBSPIQ)
- net GPIO37: now also J14.6 (Pin_6)
- net GPIO38: now reaches U8.31 (GPIO38/FSPIWP/SUBSPIWP)
- net GPIO38: now also J14.5 (Pin_5)
- net GPIO39: now reaches U8.32 (MTCK/GPIO39/CLK_OUT3/SUBSPICS1)
- net GPIO39: now also J14.4 (Pin_4)
- net GPIO40: now reaches U8.33 (MTDO/GPIO40/CLK_OUT2)
- net GPIO40: now also J14.3 (Pin_3)
- net GPIO41: now reaches U8.34 (MTDI/GPIO41/CLK_OUT1)
- net GPIO41: now also J14.2 (Pin_2)
- net GPIO42: now reaches U8.35 (MTMS/GPIO42)
- net GPIO42: now also J14.1 (Pin_1)
- net ESP_UART_RX renamed ESP_RX
- net ESP_UART_TX renamed ESP_TX
- new net Handshake2: J11.2 (Pin_2), U8.22 (GPIO14/TOUCH14/ADC2_CH3/FSPIWP/FSPIDQS/SUBSPIWP)
- new net VCC: J11.8 (Pin_8)
- no-connect marks 8 -> 6
Other:
- sheet ESP32CAM ports: added USB_RX, USB_TX; removed none
- note added: "GPIO + 3.3V Rails"
- moved on the sheet: C19, C20, C21, C22, J6

Commit message: Rev 1
Connections:
- net +3.3V: no longer J4.1
- net +5V: now also J4.1
Changed lines of the file:
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@@
   (junction (at 278.13 54.61) (diameter 0) (color 0 0 0 0)
-  )
-  (junction (at 255.27 146.812) (diameter 0) (color 0 0 0 0)
   )
   (junction (at 118.11 146.685) (diameter 0) (color 0 0 0 0)
@@
     (stroke (width 0) (type default))
   )
-  (wire (pts (xy 270.002 146.812) (xy 270.002 154.94))
-    (stroke (width 0) (type default))
-  )
   (wire (pts (xy 253.365 39.37) (xy 241.3 39.37))
     (stroke (width 0) (type default))
   )
-  (wire (pts (xy 255.27 144.145) (xy 255.27 146.812))
+  (wire (pts (xy 255.27 144.145) (xy 255.27 149.86))
     (stroke (width 0) (type default))
   )
@@
     (stroke (width 0) (type default))
   )
-  (wire (pts (xy 255.27 146.812) (xy 270.002 146.812))
-    (stroke (width 0) (type default))
-  )
   (wire (pts (xy 20.955 95.25) (xy 33.02 95.25))
     (stroke (width 0) (type default))
@@
     (stroke (width 0) (type default))
   )
-  (wire (pts (xy 255.27 146.812) (xy 255.27 149.86))
-    (stroke (width 0) (type default))
-  )
   (wire (pts (xy 195.58 121.285) (xy 195.58 115.57))
     (stroke (width 0) (type default))
@@
   )
   (wire (pts (xy 89.916 110.617) (xy 94.996 110.617))
+    (stroke (width 0) (type default))
+  )
+  (wire (pts (xy 270.002 145.669) (xy 270.002 154.94))
     (stroke (width 0) (type default))
   )
@@
         )
       )
+    )
+  )
+  (symbol (lib_id "power:+5V") (at 270.002 145.669 0) (unit 1)
+    (in_bom yes) (on_board yes) (dnp no) (fields_autoplaced)
+    (property "Reference" "#PWR0121" (at 270.002 149.479 0)
+      (effects (font (size 1.27 1.27)) hide)
+    )
+    (property "Value" "+5V" (at 270.002 141.224 0)
+      (effects (font (size 1.27 1.27)))
+    )
+    (property "Footprint" "" (at 270.002 145.669 0)
+      (effects (font (size 1.27 1.27)) hide)
+    )
+    (property "Datasheet" "" (at 270.002 145.669 0)
+      (effects (font (size 1.27 1.27)) hide)
+    )
+    (pin "1")
+    (instances
+      (project "DeltaRhoRobot"
+        (path "/cced1a6d-3dc4-42b2-93bd-998a7b4cf4e8/5eb80655-957d-4a1c-8d7d-b2e173715026"
+          (reference "#PWR0121") (unit 1)
+        )
+      )

Commit message: Rev0.1
Connections:
- net ESP_CS1: no longer J7.24 (Pin_24)
- net ESP_MISO: no longer J7.19 (Pin_19)
- net ESP_MOSI: no longer J7.21 (Pin_21)
- net ESP_SCLK: no longer J7.23 (Pin_23)
- net SCL: now also J7.28 (Pin_28)
- net SDA: now also J7.27 (Pin_27)
- net PICO_SDA: now reaches J7.3 (Pin_3)
- net PICO_SCL: now reaches J7.5 (Pin_5)
- no-connect marks 6 -> 36
Changed lines of the file:
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@@
   (junction (at 118.11 131.445) (diameter 0) (color 0 0 0 0)
   )
+  (no_connect (at 33.02 107.95))
+  (no_connect (at 33.02 82.55))
   (no_connect (at 43.18 131.445))
+  (no_connect (at 45.72 102.87))
   (no_connect (at 19.05 36.83))
+  (no_connect (at 45.72 105.41))
+  (no_connect (at 45.72 95.25))
+  (no_connect (at 45.72 72.39))
+  (no_connect (at 45.72 87.63))
+  (no_connect (at 45.72 82.55))
+  (no_connect (at 45.72 92.71))
+  (no_connect (at 33.02 87.63))
+  (no_connect (at 45.72 100.33))
+  (no_connect (at 33.02 64.77))
+  (no_connect (at 33.02 72.39))
+  (no_connect (at 241.3 59.69))
+  (no_connect (at 33.02 77.47))
+  (no_connect (at 45.72 74.93))
   (no_connect (at 64.77 138.43))
+  (no_connect (at 33.02 105.41))
+  (no_connect (at 33.02 90.17))
+  (no_connect (at 45.72 80.01))
+  (no_connect (at 45.72 107.95))
+  (no_connect (at 33.02 80.01))
+  (no_connect (at 33.02 100.33))
+  (no_connect (at 45.72 77.47))
+  (no_connect (at 33.02 110.49))
+  (no_connect (at 249.174 97.79))
+  (no_connect (at 45.72 85.09))
+  (no_connect (at 45.72 90.17))
   (no_connect (at 64.77 143.51))
   (no_connect (at 43.18 149.225))
+  (no_connect (at 33.02 92.71))
+  (no_connect (at 33.02 102.87))
+  (no_connect (at 45.72 110.49))
   (no_connect (at 64.77 146.05))
   (bus_entry (at 86.106 92.202) (size 2.54 2.54)
@@
     (stroke (width 0) (type default))
   )
-  (wire (pts (xy 253.365 39.37) (xy 241.3 39.37))
-    (stroke (width 0) (type default))
-  )
   (wire (pts (xy 255.27 144.145) (xy 255.27 149.86))
     (stroke (width 0) (type default))
@@
     (stroke (width 0) (type default))
   )
-  (wire (pts (xy 20.955 95.25) (xy 33.02 95.25))
+  (wire (pts (xy 27.432 67.31) (xy 33.02 67.31))
+    (stroke (width 0) (type default))
+  )
+  (wire (pts (xy 14.478 99.695) (xy 14.605 99.695))
     (stroke (width 0) (type default))
   )
@@
     (stroke (width 0) (type default))
   )
+  (wire (pts (xy 14.605 99.695) (xy 14.605 95.25))
+    (stroke (width 0) (type default))
+  )
   (wire (pts (xy 57.15 69.85) (xy 45.72 69.85))
     (stroke (width 0) (type default))
@@
     (stroke (width 0) (type default))
   )
-  (wire (pts (xy 253.365 41.91) (xy 241.3 41.91))
+  (wire (pts (xy 241.3 41.91) (xy 258.191 41.91))
     (stroke (width 0) (type default))
   )
@@
     (stroke (width 0) (type default))
   )
+  (wire (pts (xy 14.605 95.25) (xy 33.02 95.25))
+    (stroke (width 0) (type default))
+  )
   (wire (pts (xy 113.03 47.752) (xy 113.03 50.292))
     (stroke (width 0) (type default))
@@
     (stroke (width 0) (type default))
   )
-  (wire (pts (xy 241.3 110.49) (xy 250.19 110.49))
+  (wire (pts (xy 241.3 110.49) (xy 260.985 110.49))
     (stroke (width 0) (type default))
   )
@@
     (stroke (width 0) (type default))
   )
+  (wire (pts (xy 52.959 97.79) (xy 45.72 97.79))
+    (stroke (width 0) (type default))
+  )
   (polyline (pts (xy 72.39 118.11) (xy 104.775 118.11))
     (stroke (width 0) (type default))
@@
     (stroke (width 0) (type default))
   )
-  (wire (pts (xy 241.3 107.95) (xy 250.19 107.95))
+  (wire (pts (xy 241.3 107.95) (xy 260.985 107.95))
     (stroke (width 0) (type default))
   )
@@
     (stroke (width 0) (type default))
   )
+  (wire (pts (xy 28.575 97.79) (xy 33.02 97.79))
+    (stroke (width 0) (type default))
+  )
   (wire (pts (xy 89.916 108.077) (xy 89.916 110.617))
     (stroke (width 0) (type default))
@@
     (stroke (width 0) (type default))
   )
+  (wire (pts (xy 27.432 69.85) (xy 33.02 69.85))
+    (stroke (width 0) (type default))
+  )
   (wire (pts (xy 127.889 174.498) (xy 139.954 174.498))
     (stroke (width 0) (type default))
@@
   )
   (wire (pts (xy 143.891 62.23) (xy 149.86 62.23))
+    (stroke (width 0) (type default))
+  )
+  (wire (pts (xy 241.3 39.37) (xy 258.191 39.37))
     (stroke (width 0) (type default))
   )
@@
     (effects (font (size 1.27 1.27)) (justify right bottom))
   )
+  (label "TWI_SDA" (at 28.575 97.79 180) (fields_autoplaced)
+    (effects (font (size 1.27 1.27)) (justify right bottom))
+  )
+  (label "TWI_SCL" (at 260.985 110.49 0) (fields_autoplaced)
+    (effects (font (size 1.27 1.27)) (justify left bottom))
+  )
   (label "Handshake" (at 40.64 133.985 180) (fields_autoplaced)
     (effects (font (size 1.27 1.27)) (justify right bottom))
   )
-  (label "ESP_MISO" (at 33.02 87.63 180) (fields_autoplaced)
-    (effects (font (size 1.27 1.27)) (justify right bottom))
-  )
-  (label "ESP_SCLK" (at 33.02 92.71 180) (fields_autoplaced)
-    (effects (font (size 1.27 1.27)) (justify right bottom))
-  )
   (label "ESP_SCLK" (at 40.64 136.525 180) (fields_autoplaced)
     (effects (font (size 1.27 1.27)) (justify right bottom))
@@
     (effects (font (size 1.27 1.27)) (justify left bottom))
   )
-  (label "ESP_MOSI" (at 33.02 90.17 180) (fields_autoplaced)
-    (effects (font (size 1.27 1.27)) (justify right bottom))
-  )
   (label "USB_RX" (at 64.516 167.894 0) (fields_autoplaced)
     (effects (font (size 1.27 1.27)) (justify left bottom))
@@
     (effects (font (size 1.27 1.27)) (justify right bottom))
   )
-  (label "ESP_CS1" (at 45.72 92.71 0) (fields_autoplaced)
-    (effects (font (size 1.27 1.27)) (justify left bottom))
-  )
   (label "GPIO_15" (at 117.856 99.822 180) (fields_autoplaced)
     (effects (font (size 1.27 1.27)) (justify right bottom))
@@
     (effects (font (size 1.27 1.27)) (justify left bottom))
   )
+  (label "TWI_SCL" (at 52.959 97.79 0) (fields_autoplaced)
+    (effects (font (size 1.27 1.27)) (justify left bottom))
+  )
   (label "GPIO37" (at 85.344 59.944 180) (fields_autoplaced)
     (effects (font (size 1.27 1.27)) (justify right bottom))
@@
     (effects (font (size 1.27 1.27)) (justify left bottom))
   )
+  (label "TWI_SDA" (at 260.985 107.95 0) (fields_autoplaced)
+    (effects (font (size 1.27 1.27)) (justify left bottom))
+  )
   (label "ESP_MISO" (at 60.325 178.435 0) (fields_autoplaced)
     (effects (font (size 1.27 1.27)) (justify left bottom))
@@
     (effects (font (size 1.27 1.27)) (justify right bottom))
   )
-  (global_label "ESP_RX" (shape input) (at 253.365 41.91 0) (fields_autoplaced)
+  (global_label "ESP_RX" (shape input) (at 258.191 41.91 0) (fields_autoplaced)
     (effects (font (size 1.27 1.27)) (justify left))
-    (property "Intersheetrefs" "${INTERSHEET_REFS}" (at 263.4258 41.91 0)
+    (property "Intersheetrefs" "${INTERSHEET_REFS}" (at 268.2518 41.91 0)
       (effects (font (size 1.27 1.27)) (justify left) hide)
     )
   )
-  (global_label "ESP_TX" (shape input) (at 253.365 39.37 0) (fields_autoplaced)
+  (global_label "ESP_TX" (shape input) (at 258.191 39.37 0) (fields_autoplaced)
     (effects (font (size 1.27 1.27)) (justify left))
-    (property "Intersheetrefs" "${INTERSHEET_REFS}" (at 263.1234 39.37 0)
+    (property "Intersheetrefs" "${INTERSHEET_REFS}" (at 267.9494 39.37 0)
       (effects (font (size 1.27 1.27)) (justify left) hide)
+    )
+  )
+  (global_label "PICO_SDA" (shape input) (at 27.432 67.31 180) (fields_autoplaced)
+    (effects (font (size 1.27 1.27)) (justify right))
+    (property "Intersheetrefs" "${INTERSHEET_REFS}" (at 15.4358 67.31 0)
+      (effects (font (size 1.27 1.27)) (justify right) hide)
+    )
+  )
+  (global_label "PICO_SCL" (shape input) (at 27.432 69.85 180) (fields_autoplaced)
+    (effects (font (size 1.27 1.27)) (justify right))
+    (property "Intersheetrefs" "${INTERSHEET_REFS}" (at 15.4963 69.85 0)
+      (effects (font (size 1.27 1.27)) (justify right) hide)
     )
   )
@@
     )
   )
-  (symbol (lib_id "power:Earth") (at 20.955 95.25 0) (mirror y) (unit 1)
+  (symbol (lib_id "power:Earth") (at 14.478 99.695 0) (mirror y) (unit 1)
     (in_bom yes) (on_board yes) (dnp no) (fields_autoplaced)
-    (property "Reference" "#PWR073" (at 20.955 101.6 0)
+    (property "Reference" "#PWR073" (at 14.478 106.045 0)
       (effects (font (size 1.27 1.27)) hide)
     )
-    (property "Value" "Earth" (at 20.955 99.06 0)
+    (property "Value" "Earth" (at 14.478 103.505 0)
       (effects (font (size 1.27 1.27)) hide)
     )
-    (property "Footprint" "" (at 20.955 95.25 0)
+    (property "Footprint" "" (at 14.478 99.695 0)
       (effects (font (size 1.27 1.27)) hide)
     )
-    (property "Datasheet" "~" (at 20.955 95.25 0)
+    (property "Datasheet" "~" (at 14.478 99.695 0)
       (effects (font (size 1.27 1.27)) hide)
     )
