File: DeltaRhoRobot.kicad_sch (KiCad schematic)
At the start: 30 parts, among them J1 Conn_01x02_Socket, J2 USB_C_Receptacle_USB2.0, J3 USB_C_Receptacle_USB2.0, Q1 MBT3904DW1, SW1 CAS-120A1, U1 AP63205WU-7, U2 AMS1117-3.3

Commit message: Nearly done schematics
Parts:
- removed D1: 1N5820, Diode_THT:D_DO-201AD_P15.24mm_Horizontal, symbol Diode:1N5820
- added C5: .1uF, symbol Device:C
- added Q3: STB55NF06T4, Package_TO_SOT_SMD:TO-263-2, symbol Device:Q_NMOS_Depletion_GDS
- added R14: 1K, symbol Device:R_US
- added R32: 68k, Resistor_SMD:R_0402_1005Metric, symbol Device:R_US
- added SW2: SW_Push, Button_Switch_SMD:SW_SPST_PTS645, symbol Switch:SW_Push
- C4: value C_Small -> 10uF
- SW1: footprint Button_Switch_SMD:Nidec_Copal_CAS-120A -> switch185:1825232-1_TEC; symbol Switch:SW_Nidec_CAS-120A1 -> Switch:SW_SPDT
- U2: footprint Package_SO:SOIC-8_3.9x4.9mm_P1.27mm -> Package_TO_SOT_SMD:SOT-223-3_TabPin2
- renumbered C5 to C6
Connections:
- net +3.3V: now also R14.1
- net Earth: now also SW1.3 (C), C5.2, SW2.2
- net VCC: now also Q3.2 (D), R32.1
- net at C3.1, U1.2 (EN), U1.3 (IN)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: now also D2.3, Q3.3 (S); no longer SW1.3 (A)
- net at SW1.1 (A): now also R32.2
- net at SW1.2 (B): now also Q3.1 (G); no longer D2.3
- new net ESP_PU: C5.1, R14.2, SW2.1
- no-connect marks 5 -> 4
Other:
- sheet ESP32-S3-WROOM-1 ports: added ESP_PU; removed none
- sheet Pico ports: added Pico_PU; removed none
- note added: "Reset chips"
- moved on the sheet: C1, C2, C3, C4, L1, SW1, U1, U2

Commit message: Much much more progress
Parts:
- removed R11: 220, Resistor_SMD:R_0402_1005Metric, symbol Device:R_US
- added C34: .1uf, Capacitor_SMD:C_0402_1005Metric, symbol Device:C
- C2: footprint Capacitor_SMD:C_0402_1005Metric -> Capacitor_SMD:C_Elec_6.3x5.8
- C5: footprint (none) -> Capacitor_SMD:C_0402_1005Metric
- R14: footprint (none) -> Resistor_SMD:R_0402_1005Metric
- renumbered SW2 to RST1
Connections:
- net Earth: now also C34.2
- net VCC: now also C3.1, D2.3, Q3.3 (S), U1.2 (EN), U1.3 (IN), U2.3 (VI), C34.1; no longer J1.2 (Pin_2), Q3.2 (D), R32.1
- net at Q1.3 (C2), R10.2: now also Q1.6 (C1)
- net ESP_PICO_UART_RX renamed ESP_RX
- net ESP_PICO_UART_TX renamed ESP_TX
- new net VS: J1.2 (Pin_2), Q3.2 (D), R32.1
Other:
- sheet ESP32-S3-WROOM-1 ports: added none; removed ESP_UART_RX, ESP_UART_TX
- sheet Pico ports: added none; removed PICO_UART_RX, PICO_UART_TX
- moved on the sheet: D2, R10

Commit message: Rev 1
Parts:
- removed R3, R9: 1M, Resistor_SMD:R_0402_1005Metric, symbol Device:R_US
- C3: footprint Capacitor_SMD:C_0402_1005Metric -> Capacitor_SMD:C_0805_2012Metric
Connections:
- net Earth: now also J2.S1 (SHIELD), J3.S1 (SHIELD)
Changed lines of the file:
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@@
-    (stroke (width 0) (type default))
-  )
-  (wire (pts (xy 25.4 73.66) (xy 25.4 74.93))
     (stroke (width 0) (type default))
   )
@@
     (stroke (width 0) (type default))
   )
-  (wire (pts (xy 25.4 66.04) (xy 25.4 65.405))
+  (wire (pts (xy 25.4 65.405) (xy 25.4 74.93))
     (stroke (width 0) (type default))
   )
@@
     (stroke (width 0) (type default))
   )
-  (wire (pts (xy 24.13 133.985) (xy 24.13 133.35))
-    (stroke (width 0) (type default))
-  )
   (wire (pts (xy 189.23 115.57) (xy 199.39 115.57))
     (stroke (width 0) (type default))
@@
     (stroke (width 0) (type default))
   )
-  (wire (pts (xy 24.13 142.875) (xy 24.13 141.605))
+  (wire (pts (xy 24.13 133.35) (xy 24.13 142.875))
     (stroke (width 0) (type default))
   )
@@
         (path "/cced1a6d-3dc4-42b2-93bd-998a7b4cf4e8"
           (reference "U2") (unit 1)
-        )
-      )
-    )
-  )
-  (symbol (lib_id "Device:R_US") (at 24.13 137.795 0) (unit 1)
-    (in_bom yes) (on_board yes) (dnp no) (fields_autoplaced)
-    (property "Reference" "R9" (at 26.67 136.525 0)
-      (effects (font (size 1.27 1.27)) (justify left))
-    )
-    (property "Value" "1M" (at 26.67 139.065 0)
-      (effects (font (size 1.27 1.27)) (justify left))
-    )
-    (property "Footprint" "Resistor_SMD:R_0402_1005Metric" (at 25.146 138.049 90)
-      (effects (font (size 1.27 1.27)) hide)
-    )
-    (property "Datasheet" "~" (at 24.13 137.795 0)
-      (effects (font (size 1.27 1.27)) hide)
-    )
-    (pin "1")
-    (pin "2")
-    (instances
-      (project "DeltaRhoRobot"
-        (path "/cced1a6d-3dc4-42b2-93bd-998a7b4cf4e8"
-          (reference "R9") (unit 1)
         )
       )
@@
     )
   )
-  (symbol (lib_id "Device:R_US") (at 25.4 69.85 0) (unit 1)
-    (in_bom yes) (on_board yes) (dnp no) (fields_autoplaced)
-    (property "Reference" "R3" (at 27.94 68.58 0)
-      (effects (font (size 1.27 1.27)) (justify left))
-    )
-    (property "Value" "1M" (at 27.94 71.12 0)
-      (effects (font (size 1.27 1.27)) (justify left))
-    )
-    (property "Footprint" "Resistor_SMD:R_0402_1005Metric" (at 26.416 70.104 90)
-      (effects (font (size 1.27 1.27)) hide)
-    )
-    (property "Datasheet" "~" (at 25.4 69.85 0)
-      (effects (font (size 1.27 1.27)) hide)
-    )
-    (pin "1")
-    (pin "2")
-    (instances
-      (project "DeltaRhoRobot"
-        (path "/cced1a6d-3dc4-42b2-93bd-998a7b4cf4e8"
-          (reference "R3") (unit 1)
-        )
-      )
-    )
-  )
   (symbol (lib_id "Connector:USB_C_Receptacle_USB2.0") (at 31.75 110.49 0) (unit 1)
     (in_bom yes) (on_board yes) (dnp no) (fields_autoplaced)
@@
       (effects (font (size 1.27 1.27)) (justify left))
     )
-    (property "Footprint" "Capacitor_SMD:C_0402_1005Metric" (at 163.83 66.675 0)
-      (effects (font (size 1.27 1.27)) hide)
-    )
+    (property "Footprint" "Capacitor_SMD:C_0805_2012Metric" (at 163.83 66.675 0)
+      (effects (font (size 1.27 1.27)) hide)
+    )

Commit message: Rev0.1
Parts:
- added H1, H2, H3, H4: MountingHole_Pad, MountingHole:MountingHole_3.2mm_M3_ISO14580_Pad_TopOnly, symbol Mechanical:MountingHole_Pad
- added TP1: TestPoint_2Pole, TestPoint:TestPoint_2Pads_Pitch2.54mm_Drill0.8mm, symbol Connector:TestPoint_2Pole
Connections:
- net ESP_RX: now also TP1.1
- net ESP_TX: now also TP1.2
- no-connect marks 4 -> 8
Changed lines of the file:
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@@
   (junction (at 125.222 170.18) (diameter 0) (color 0 0 0 0)
   )
+  (no_connect (at 94.107 109.474))
   (no_connect (at 48.26 55.245))
+  (no_connect (at 94.107 102.616))
   (no_connect (at 46.99 125.73))
+  (no_connect (at 93.98 90.043))
+  (no_connect (at 93.98 95.885))
   (no_connect (at 48.26 57.785))
   (no_connect (at 46.99 123.19))
@@
     (stroke (width 0) (type default))
   )
-  (wire (pts (xy 111.76 24.13) (xy 111.76 26.035))
+  (wire (pts (xy 111.76 23.749) (xy 111.76 26.035))
     (stroke (width 0) (type default))
   )
@@
     (stroke (width 0) (type default))
   )
+  (wire (pts (xy 95.504 135.255) (xy 104.013 135.255))
+    (stroke (width 0) (type default))
+  )
   (wire (pts (xy 65.405 114.935) (xy 65.405 118.11))
     (stroke (width 0) (type default))
@@
   )
   (wire (pts (xy 236.855 39.37) (xy 236.855 51.435))
+    (stroke (width 0) (type default))
+  )
+  (wire (pts (xy 124.079 135.255) (xy 114.173 135.255))
     (stroke (width 0) (type default))
   )
@@
     )
   )
+  (global_label "ESP_RX" (shape input) (at 124.079 135.255 0) (fields_autoplaced)
+    (effects (font (size 1.27 1.27)) (justify left))
+    (property "Intersheetrefs" "${INTERSHEET_REFS}" (at 134.1398 135.255 0)
+      (effects (font (size 1.27 1.27)) (justify left) hide)
+    )
+  )
+  (global_label "ESP_TX" (shape input) (at 95.504 135.255 180) (fields_autoplaced)
+    (effects (font (size 1.27 1.27)) (justify right))
+    (property "Intersheetrefs" "${INTERSHEET_REFS}" (at 85.7456 135.255 0)
+      (effects (font (size 1.27 1.27)) (justify right) hide)
+    )
+  )
   (symbol (lib_id "Regulator_Linear:AMS1117-3.3") (at 179.07 60.96 0) (unit 1)
     (in_bom yes) (on_board yes) (dnp no) (fields_autoplaced)
@@
     )
   )
+  (symbol (lib_id "Mechanical:MountingHole_Pad") (at 94.107 106.934 0) (unit 1)
+    (in_bom yes) (on_board yes) (dnp no) (fields_autoplaced)
+    (property "Reference" "H4" (at 96.647 104.394 0)
+      (effects (font (size 1.27 1.27)) (justify left))
+    )
+    (property "Value" "MountingHole_Pad" (at 96.647 106.934 0)
+      (effects (font (size 1.27 1.27)) (justify left))
+    )
+    (property "Footprint" "MountingHole:MountingHole_3.2mm_M3_ISO14580_Pad_TopOnly" (at 94.107 106.934 0)
+      (effects (font (size 1.27 1.27)) hide)
+    )
+    (property "Datasheet" "~" (at 94.107 106.934 0)
+      (effects (font (size 1.27 1.27)) hide)
+    )
+    (pin "1")
+    (instances
+      (project "DeltaRhoRobot"
+        (path "/cced1a6d-3dc4-42b2-93bd-998a7b4cf4e8"
+          (reference "H4") (unit 1)
+        )
+      )
+    )
+  )
+  (symbol (lib_id "Connector:TestPoint_2Pole") (at 109.093 135.255 180) (unit 1)
+    (in_bom yes) (on_board yes) (dnp no) (fields_autoplaced)
+    (property "Reference" "TP1" (at 109.093 130.175 0)
+      (effects (font (size 1.27 1.27)))
+    )
+    (property "Value" "TestPoint_2Pole" (at 109.093 132.715 0)
+      (effects (font (size 1.27 1.27)))
+    )
+    (property "Footprint" "TestPoint:TestPoint_2Pads_Pitch2.54mm_Drill0.8mm" (at 109.093 135.255 0)
+      (effects (font (size 1.27 1.27)) hide)
+    )
+    (property "Datasheet" "~" (at 109.093 135.255 0)
+      (effects (font (size 1.27 1.27)) hide)
+    )
+    (pin "2")
+    (pin "1")
+    (instances
+      (project "DeltaRhoRobot"
+        (path "/cced1a6d-3dc4-42b2-93bd-998a7b4cf4e8"
+          (reference "TP1") (unit 1)
+        )
+      )
+    )
+  )
   (symbol (lib_id "Device:C_Small") (at 199.39 121.92 0) (unit 1)
     (in_bom yes) (on_board yes) (dnp no) (fields_autoplaced)
@@
     )
   )
-  (symbol (lib_id "power:VS") (at 111.76 24.13 0) (unit 1)
-    (in_bom yes) (on_board yes) (dnp no) (fields_autoplaced)
-    (property "Reference" "#PWR0107" (at 106.68 27.94 0)
-      (effects (font (size 1.27 1.27)) hide)
-    )
-    (property "Value" "VS" (at 111.76 19.05 0)
-      (effects (font (size 1.27 1.27)))
-    )
-    (property "Footprint" "" (at 111.76 24.13 0)
-      (effects (font (size 1.27 1.27)) hide)
-    )
-    (property "Datasheet" "" (at 111.76 24.13 0)
+  (symbol (lib_id "power:VS") (at 111.76 23.749 0) (unit 1)
+    (in_bom yes) (on_board yes) (dnp no) (fields_autoplaced)
+    (property "Reference" "#PWR0107" (at 106.68 27.559 0)
+      (effects (font (size 1.27 1.27)) hide)
+    )
+    (property "Value" "VS" (at 111.76 18.669 0)
+      (effects (font (size 1.27 1.27)))
+    )
+    (property "Footprint" "" (at 111.76 23.749 0)
+      (effects (font (size 1.27 1.27)) hide)
+    )
+    (property "Datasheet" "" (at 111.76 23.749 0)
       (effects (font (size 1.27 1.27)) hide)
     )
@@
         (path "/cced1a6d-3dc4-42b2-93bd-998a7b4cf4e8"
           (reference "#PWR01") (unit 1)
+        )
+      )
+    )
+  )
+  (symbol (lib_id "Mechanical:MountingHole_Pad") (at 94.107 100.076 0) (unit 1)
+    (in_bom yes) (on_board yes) (dnp no) (fields_autoplaced)
+    (property "Reference" "H3" (at 96.647 97.536 0)
+      (effects (font (size 1.27 1.27)) (justify left))
+    )
+    (property "Value" "MountingHole_Pad" (at 96.647 100.076 0)
+      (effects (font (size 1.27 1.27)) (justify left))
+    )
+    (property "Footprint" "MountingHole:MountingHole_3.2mm_M3_ISO14580_Pad_TopOnly" (at 94.107 100.076 0)
+      (effects (font (size 1.27 1.27)) hide)
+    )
+    (property "Datasheet" "~" (at 94.107 100.076 0)
+      (effects (font (size 1.27 1.27)) hide)
+    )
+    (pin "1")
+    (instances
+      (project "DeltaRhoRobot"
+        (path "/cced1a6d-3dc4-42b2-93bd-998a7b4cf4e8"
+          (reference "H3") (unit 1)
         )
       )
@@
     )
   )
+  (symbol (lib_id "Mechanical:MountingHole_Pad") (at 93.98 93.345 0) (unit 1)
+    (in_bom yes) (on_board yes) (dnp no) (fields_autoplaced)
+    (property "Reference" "H2" (at 96.52 90.805 0)
+      (effects (font (size 1.27 1.27)) (justify left))
+    )
+    (property "Value" "MountingHole_Pad" (at 96.52 93.345 0)
+      (effects (font (size 1.27 1.27)) (justify left))
+    )
+    (property "Footprint" "MountingHole:MountingHole_3.2mm_M3_ISO14580_Pad_TopOnly" (at 93.98 93.345 0)
+      (effects (font (size 1.27 1.27)) hide)
+    )
+    (property "Datasheet" "~" (at 93.98 93.345 0)
+      (effects (font (size 1.27 1.27)) hide)
+    )
+    (pin "1")
+    (instances
+      (project "DeltaRhoRobot"
+        (path "/cced1a6d-3dc4-42b2-93bd-998a7b4cf4e8"
+          (reference "H2") (unit 1)
+        )
+      )
+    )
+  )
   (symbol (lib_id "Connector:Conn_01x02_Socket") (at 94.615 28.575 180) (unit 1)
     (in_bom yes) (on_board yes) (dnp no) (fields_autoplaced)
@@
         )
       )
+    )
+  )
+  (symbol (lib_id "Mechanical:MountingHole_Pad") (at 93.98 87.503 0) (unit 1)
+    (in_bom yes) (on_board yes) (dnp no) (fields_autoplaced)
+    (property "Reference" "H1" (at 96.52 84.963 0)
+      (effects (font (size 1.27 1.27)) (justify left))
+    )
+    (property "Value" "MountingHole_Pad" (at 96.52 87.503 0)
+      (effects (font (size 1.27 1.27)) (justify left))
+    )
+    (property "Footprint" "MountingHole:MountingHole_3.2mm_M3_ISO14580_Pad_TopOnly" (at 93.98 87.503 0)
+      (effects (font (size 1.27 1.27)) hide)
+    )
+    (property "Datasheet" "~" (at 93.98 87.503 0)
+      (effects (font (size 1.27 1.27)) hide)
+    )
+    (pin "1")
+    (instances
+      (project "DeltaRhoRobot"
+        (path "/cced1a6d-3dc4-42b2-93bd-998a7b4cf4e8"
+          (reference "H1") (unit 1)
+        )
+      )
