File: _autosave-ESP.kicad_sch (KiCad schematic)
At the start: 39 parts, among them J5 JST-XH, P1 B6B-ZRLFSN, P2 B6B-ZRLFSN, P3 B6B-ZRLFSN, P4 B6B-ZRLFSN, P5 B6B-ZRLFSN, P6 B6B-ZRLFSN, U14 W25Q16JVS, U3 DRV8835DSSR, U4 RP2040, U5 DRV8835DSSR, U6 DRV8835DSSR, Y1 ABM8-272-T3

Commit message: Rev 2 PCB
Parts:
- TP2: footprint (none) -> TestPoint:TestPoint_Pad_D1.5mm
Changed lines of the file:
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@@
 			)
 		)
-		(property "Footprint" ""
+		(property "Footprint" "TestPoint:TestPoint_Pad_D1.5mm"
 			(at 105.41 154.94 0)
 			(effects
