File: ICM_20984.kicad_sch (KiCad schematic)
At the start: 17 parts, among them Q1 BSS138, Q2 BSS138, U3 ICM-42688-P, U4 LIS3MDL, U5 MIC5366-1.8YC5-TR

Commit message: Commit message
Parts:
- C13: LCSC Part # C15195 -> C15525
